File: hw/sch_pcb/USTTHUNDERMILLPCB01A/CPU.kicad_sch (KiCad schematic)
At the start: 28 parts, among them J4 HEADER_2x03, J5 SM08B-GHS-TB, J6 SM06B-GHS-TB, U7 SHT31, U8 ATMEGA1284P-AU, U9 AT24CS64-SSHM, Y1 16MHz

Commit message: Edit PCB
Parts:
- C15, C17: value 100nF -> x pF
Changed lines of the file:
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@@
       (effects (font (size 1.27 1.27)) (justify left))
     )
-    (property "Value" "100nF" (id 1) (at 51.181 67.818 0)
+    (property "Value" "x pF" (id 1) (at 51.181 67.818 0)
       (effects (font (size 1.27 1.27)) (justify left))
     )
@@
       (effects (font (size 1.27 1.27)) (justify left))
     )
-    (property "Value" "100nF" (id 1) (at 77.851 67.818 0)
+    (property "Value" "x pF" (id 1) (at 77.851 67.818 0)
       (effects (font (size 1.27 1.27)) (justify left))
     )
