File: hw/sch_pcb/USTTHUNDERMILLPCB01A/CPU.kicad_sch (KiCad schematic)
At the start: 32 parts, among them J3 HEADER_2x01_PARALLEL, J4 HEADER_2x03, J5 SM08B-GHS-TB, J6 SM06B-GHS-TB, U7 SHT31, U8 ATMEGA1284P-AU, U9 AT24CS64-SSHM, Y1 16MHz

Commit message: Edit
Parts:
- C12, C13, C14, C15, C16, C17, C18, C19, C20, C23, C24: UST_ID 5c70984712875079b91f8b4c -> (none)
- C21: UST_ID 5c70984812875079b91f8bbd -> (none)
- C22: UST_ID 5c70984712875079b91f8b52 -> (none)
- D4: UST_ID 5c70984712875079b91f8b67 -> (none)
- J6: UST_ID (none) -> 5fa0f70212875025b3977932
- R14: UST_ID 5c70984612875079b91f899f -> (none)
- R15: UST_ID 5c70984612875079b91f8990 -> (none)
- R18: UST_ID 5c70984512875079b91f896b -> (none)
- Y1: UST_ID 5c70984712875079b91f8b10 -> (none)
Connections:
- net at R17.2: now also J6.3; no longer J6.2
- net at R16.2: now also J6.2; no longer J6.3
Other:
- moved on the sheet: R16, R17

Commit message: Edit PCB
Parts:
- removed C22: 4u7, Mlab_R:SMD-0805, symbol DATALOGGER01A-rescue:C-device
- removed J3: HEADER_2x01_PARALLEL, Mlab_Pin_Headers:Straight_2x01, symbol DATALOGGER01A-rescue:HEADER_2x01_PARALLEL-MLAB_HEADER
- removed R18: 0R, Mlab_R:SMD-0805, symbol DATALOGGER01A-rescue:R-device
- removed R19: -, Mlab_R:SMD-0805, symbol DATALOGGER01A-rescue:R-device
- C11, C12, C13, C14, C15, C16, C17, C18, C19, C20, C23, C24: footprint Mlab_R:SMD-0805 -> Capacitor_SMD:C_0603_1608Metric
- C21: footprint Mlab_R:SMD-0805 -> Capacitor_SMD:C_0805_2012Metric
- D4: value HLMP-K150+FIX-LED-313 -> RED; footprint Mlab_D:FIX-LED-313 -> LED_SMD:LED_0603_1608Metric
- R12, R13, R14, R15: footprint Mlab_R:SMD-0805 -> Resistor_SMD:R_0603_1608Metric
Connections:
- net GND: now also U9.7 (WP)

Commit message: Edit PCB
Parts:
- removed Y1: 16MHz, Mlab_XTAL:Crystal_HC49-U_Vertical, symbol Device:Crystal
- added Y1: 16MHz, Mlab_XTAL:Crystal SMD CFPX-180, symbol Device:Crystal_GND24
- J4: footprint Mlab_Pin_Headers:Straight_2x03 -> Mlab_Pin_Headers:SMD_2x03
- L1: footprint Mlab_R:SMD-1210 -> Inductor_SMD:L_1210_3225Metric
Connections:
- net GND: now also Y1.2, Y1.4
- net at C15.1, U8.7 (XTAL2): now also Y1.1
- net at C17.1, U8.8 (XTAL1): now also Y1.3
Changed lines of the file:
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@@
   (junction (at 62.23 20.955) (diameter 1.016) (color 0 0 0 0))
   (junction (at 64.77 168.275) (diameter 1.016) (color 0 0 0 0))
+  (junction (at 71.12 65.405) (diameter 1.016) (color 0 0 0 0))
   (junction (at 74.93 59.055) (diameter 1.016) (color 0 0 0 0))
   (junction (at 115.57 69.215) (diameter 1.016) (color 0 0 0 0))
@@
     (stroke (width 0) (type solid) (color 0 0 0 0))
   )
+  (wire (pts (xy 59.69 59.055) (xy 62.23 59.055))
+    (stroke (width 0) (type solid) (color 0 0 0 0))
+  )
   (wire (pts (xy 59.69 71.755) (xy 59.69 70.485))
     (stroke (width 0) (type solid) (color 0 0 0 0))
@@
     (stroke (width 0) (type solid) (color 0 0 0 0))
   )
-  (wire (pts (xy 66.04 59.055) (xy 59.69 59.055))
-    (stroke (width 0) (type solid) (color 0 0 0 0))
-  )
-  (wire (pts (xy 74.93 59.055) (xy 73.66 59.055))
+  (wire (pts (xy 66.04 52.07) (xy 66.04 53.975))
+    (stroke (width 0) (type solid) (color 0 0 0 0))
+  )
+  (wire (pts (xy 66.04 52.07) (xy 71.12 52.07))
+    (stroke (width 0) (type solid) (color 0 0 0 0))
+  )
+  (wire (pts (xy 66.04 64.135) (xy 66.04 65.405))
+    (stroke (width 0) (type solid) (color 0 0 0 0))
+  )
+  (wire (pts (xy 66.04 65.405) (xy 71.12 65.405))
+    (stroke (width 0) (type solid) (color 0 0 0 0))
+  )
+  (wire (pts (xy 69.85 59.055) (xy 74.93 59.055))
+    (stroke (width 0) (type solid) (color 0 0 0 0))
+  )
+  (wire (pts (xy 71.12 52.07) (xy 71.12 65.405))
+    (stroke (width 0) (type solid) (color 0 0 0 0))
+  )
+  (wire (pts (xy 71.12 65.405) (xy 71.12 71.755))
     (stroke (width 0) (type solid) (color 0 0 0 0))
   )
@@
     (pin "1")
   )
+  (symbol (lib_id "power:GND") (at 71.12 71.755 0) (unit 1)
+    (in_bom yes) (on_board yes)
+    (property "Reference" "#PWR0101" (id 0) (at 71.12 78.105 0)
+      (effects (font (size 1.27 1.27)) hide)
+    )
+    (property "Value" "GND" (id 1) (at 71.247 76.1492 0))
+    (property "Footprint" "" (id 2) (at 71.12 71.755 0)
+      (effects (font (size 1.27 1.27)) hide)
+    )
+    (property "Datasheet" "" (id 3) (at 71.12 71.755 0)
+      (effects (font (size 1.27 1.27)) hide)
+    )
+    (pin "1")
+  )
   (symbol (lib_id "power:GND") (at 74.93 71.755 0) (unit 1)
     (in_bom yes) (on_board yes)
@@
     (property "Reference" "L1" (id 0) (at 52.07 16.129 90))
     (property "Value" "10uH - LQH32CN100K23L" (id 1) (at 52.07 18.4404 90))
-    (property "Footprint" "Mlab_R:SMD-1210" (id 2) (at 52.07 20.955 0)
+    (property "Footprint" "Inductor_SMD:L_1210_3225Metric" (id 2) (at 52.07 20.955 0)
       (effects (font (size 1.27 1.27)) hide)
     )
@@
   (symbol (lib_id "DATALOGGER01A-rescue:C-device") (at 59.69 66.675 0) (unit 1)
     (in_bom yes) (on_board yes)
-    (property "Reference" "C15" (id 0) (at 62.611 65.5066 0)
-      (effects (font (size 1.27 1.27)) (justify left))
-    )
-    (property "Value" "100nF" (id 1) (at 62.611 67.818 0)
+    (property "Reference" "C15" (id 0) (at 52.451 65.5066 0)
+      (effects (font (size 1.27 1.27)) (justify left))
+    )
+    (property "Value" "100nF" (id 1) (at 51.181 67.818 0)
       (effects (font (size 1.27 1.27)) (justify left))
     )
@@
     (pin "2")
   )
-  (symbol (lib_id "Device:Crystal") (at 69.85 59.055 0) (unit 1)
-    (in_bom yes) (on_board yes)
-    (property "Reference" "Y1" (id 0) (at 69.85 52.2478 0))
-    (property "Value" "16MHz" (id 1) (at 69.85 54.5592 0))
-    (property "Footprint" "Mlab_XTAL:Crystal_HC49-U_Vertical" (id 2) (at 69.85 59.055 0)
-      (effects (font (size 1.27 1.27)) hide)
-    )
-    (property "Datasheet" "~" (id 3) (at 69.85 59.055 0)
-      (effects (font (size 1.27 1.27)) hide)
-    )
-    (property "USD_ID" "" (id 4) (at 69.85 59.055 0)
-      (effects (font (size 1.27 1.27)) hide)
-    )
-    (property "UST_ID" "" (id 5) (at 69.85 59.055 0)
-      (effects (font (size 1.27 1.27)) hide)
-    )
-    (pin "1")
-    (pin "2")
+  (symbol (lib_id "Device:Crystal_GND24") (at 66.04 59.055 0) (unit 1)
+    (in_bom yes) (on_board yes)
+    (property "Reference" "Y1" (id 0) (at 72.1361 53.2141 0)
+      (effects (font (size 1.27 1.27)) (justify left))
+    )
+    (property "Value" "16MHz" (id 1) (at 72.1361 55.5128 0)
+      (effects (font (size 1.27 1.27)) (justify left))
+    )
+    (property "Footprint" "Mlab_XTAL:Crystal SMD CFPX-180" (id 2) (at 66.04 59.055 0)
+      (effects (font (size 1.27 1.27)) hide)
+    )
+    (property "Datasheet" "LFXTAL035264REEL" (id 3) (at 66.04 59.055 0)
+      (effects (font (size 1.27 1.27)) hide)
+    )
+    (pin "1")
+    (pin "2")
+    (pin "3")
+    (pin "4")
   )
   (symbol (lib_id "DATALOGGER01A-rescue:HEADER_2x03-MLAB_HEADER") (at 148.59 158.115 0) (unit 1)
@@
       (effects (font (size 1.524 1.524)) hide)
     )
-    (property "Footprint" "Mlab_Pin_Headers:Straight_2x03" (id 2) (at 148.59 155.575 0)
+    (property "Footprint" "Mlab_Pin_Headers:SMD_2x03" (id 2) (at 148.59 155.575 0)
       (effects (font (size 1.524 1.524)) hide)
     )

Commit message: Uprava PCB
Parts:
- added D3, D5: RED, LED_SMD:LED_0603_1608Metric, symbol DATALOGGER01A-rescue:LED-device
- added R18, R5: 2k2, Resistor_SMD:R_0603_1608Metric, symbol DATALOGGER01A-rescue:R-device
- added SW1: SW_Push, Button_Switch_SMD:SW_SPST_B3S-1000, symbol Switch:SW_Push
Connections:
- net GND: now also D3.1 (K), D5.1 (K), SW1.1
- net TX1: now reaches J5.6
- net TX1: now also U8.12 ((PCINT27/TXD1/INT1)PD3)
- net RX1: now reaches J5.7
- net RX1: now also U8.11 ((PCINT26/RXD1/INT0)PD2)
- net LED: no longer names the net of U8.26 ((PCINT23/TOSC2)PC7)
- net LED: no longer R15.2
- new net: D3.2 (A), R5.1
- new net: D5.2 (A), R18.1
- new net BTN: SW1.2
- new net LED_1: R15.2
- new net LED_2: R5.2
- new net LED_3: R18.2
- no-connect marks 31 -> 27
