File: hw/sch_pcb/USTTHUNDERMILLPCB01A/CPU.kicad_sch (KiCad schematic)
At the start: 33 parts, among them J4 HEADER_2x03, J5 SM08B-GHS-TB, J6 SM06B-GHS-TB, SW1 SW_Push, U7 SHT31, U8 ATMEGA1284P-AU, U9 AT24CS64-SSHM, Y1 16MHz

Commit message: Edit PCB
Connections:
- net BTN: now also U8.24 ((PCINT21/TDI)PC5)
- net COUNT_1_PCFO: now also U8.21 ((PCINT18/TCK)PC2)
- net LED_1: now also U8.14 ((PCINT294/OC1A)PD5)
- net LED_2: now also U8.15 ((PCINT30/OC2B/ICP)PD6)
- net LED_3: now also U8.16 ((PCINT31/OC2A)PD7)
- no-connect marks 27 -> 23
Other:
- moved on the sheet: SW1
Changed lines of the file:
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@@
-(kicad_sch (version 20210621) (generator eeschema)
+(kicad_sch (version 20210406) (generator eeschema)
   (paper "A4")
   (junction (at 17.78 20.955) (diameter 1.016) (color 0 0 0 0))
@@
   (no_connect (at 172.72 69.215))
   (no_connect (at 172.72 71.755))
-  (no_connect (at 172.72 89.535))
-  (no_connect (at 172.72 97.155))
   (no_connect (at 172.72 99.695))
+  (no_connect (at 172.72 102.235))
   (no_connect (at 172.72 117.475))
-  (no_connect (at 172.72 120.015))
-  (no_connect (at 172.72 122.555))
-  (no_connect (at 172.72 125.095))
   (no_connect (at 224.79 127.635))
   (no_connect (at 224.79 130.175))
@@
     (stroke (width 0) (type solid) (color 0 0 0 0))
   )
-  (wire (pts (xy 172.72 92.075) (xy 175.895 92.075))
-    (stroke (width 0) (type solid) (color 0 0 0 0))
-  )
-  (wire (pts (xy 172.72 94.615) (xy 175.895 94.615))
+  (wire (pts (xy 172.72 89.535) (xy 175.26 89.535))
+    (stroke (width 0) (type solid) (color 0 0 0 0))
+  )
+  (wire (pts (xy 172.72 92.075) (xy 175.26 92.075))
+    (stroke (width 0) (type solid) (color 0 0 0 0))
+  )
+  (wire (pts (xy 172.72 94.615) (xy 175.26 94.615))
+    (stroke (width 0) (type solid) (color 0 0 0 0))
+  )
+  (wire (pts (xy 172.72 97.155) (xy 175.26 97.155))
     (stroke (width 0) (type solid) (color 0 0 0 0))
   )
@@
     (stroke (width 0) (type solid) (color 0 0 0 0))
   )
-  (wire (pts (xy 220.345 137.795) (xy 224.79 137.795))
-    (stroke (width 0) (type solid) (color 0 0 0 0))
-  )
-  (wire (pts (xy 220.98 140.335) (xy 224.79 140.335))
+  (wire (pts (xy 172.72 120.015) (xy 175.26 120.015))
+    (stroke (width 0) (type solid) (color 0 0 0 0))
+  )
+  (wire (pts (xy 172.72 122.555) (xy 175.26 122.555))
+    (stroke (width 0) (type solid) (color 0 0 0 0))
+  )
+  (wire (pts (xy 172.72 125.095) (xy 175.26 125.095))
+    (stroke (width 0) (type solid) (color 0 0 0 0))
+  )
+  (wire (pts (xy 175.26 88.265) (xy 175.26 89.535))
+    (stroke (width 0) (type solid) (color 0 0 0 0))
+  )
+  (wire (pts (xy 175.26 93.345) (xy 175.26 94.615))
+    (stroke (width 0) (type solid) (color 0 0 0 0))
+  )
+  (wire (pts (xy 222.25 137.795) (xy 224.79 137.795))
+    (stroke (width 0) (type solid) (color 0 0 0 0))
+  )
+  (wire (pts (xy 222.25 140.335) (xy 224.79 140.335))
     (stroke (width 0) (type solid) (color 0 0 0 0))
   )
@@
     (stroke (width 0) (type solid) (color 0 0 0 0))
   )
+  (wire (pts (xy 223.52 38.735) (xy 223.52 41.275))
+    (stroke (width 0) (type solid) (color 0 0 0 0))
+  )
   (wire (pts (xy 224.79 125.095) (xy 222.25 125.095))
     (stroke (width 0) (type solid) (color 0 0 0 0))
@@
   )
   (wire (pts (xy 231.14 80.645) (xy 231.14 90.805))
-    (stroke (width 0) (type solid) (color 0 0 0 0))
-  )
-  (wire (pts (xy 232.41 38.735) (xy 232.41 41.275))
     (stroke (width 0) (type solid) (color 0 0 0 0))
   )
@@
     (effects (font (size 1.524 1.524)) (justify left bottom))
   )
-  (label "PA0" (at 175.26 38.735 0)
-    (effects (font (size 1.524 1.524)) (justify left bottom))
-  )
-  (label "PA1" (at 175.26 41.275 0)
-    (effects (font (size 1.524 1.524)) (justify left bottom))
-  )
   (label "PB5" (at 175.26 74.295 0)
     (effects (font (size 1.524 1.524)) (justify left bottom))
@@
     (effects (font (size 1.524 1.524)) (justify left bottom))
   )
+  (label "TIMEPULSE" (at 175.26 92.075 0)
+    (effects (font (size 1.524 1.524)) (justify left bottom))
+  )
+  (label "BTN" (at 175.26 97.155 0)
+    (effects (font (size 1.27 1.27)) (justify left bottom))
+  )
   (label "RX0" (at 175.26 107.315 0)
     (effects (font (size 1.524 1.524)) (justify left bottom))
@@
     (effects (font (size 1.524 1.524)) (justify left bottom))
   )
-  (label "COUNT_1_PCFO" (at 175.895 89.535 0)
-    (effects (font (size 1.27 1.27)) (justify left bottom))
-  )
-  (label "TIMEPULSE" (at 175.895 92.075 0)
-    (effects (font (size 1.524 1.524)) (justify left bottom))
-  )
-  (label "COUNT_2" (at 175.895 94.615 0)
-    (effects (font (size 1.27 1.27)) (justify left bottom))
-  )
-  (label "BTN" (at 175.895 97.155 0)
-    (effects (font (size 1.27 1.27)) (justify left bottom))
-  )
-  (label "LED_1" (at 176.53 120.015 0)
-    (effects (font (size 1.524 1.524)) (justify left bottom))
-  )
-  (label "LED_2" (at 176.53 122.555 0)
-    (effects (font (size 1.524 1.524)) (justify left bottom))
-  )
-  (label "LED_3" (at 176.53 125.095 0)
-    (effects (font (size 1.524 1.524)) (justify left bottom))
-  )
-  (label "TX1" (at 220.345 137.795 180)
-    (effects (font (size 1.524 1.524)) (justify right bottom))
-  )
-  (label "RX1" (at 220.98 140.335 180)
-    (effects (font (size 1.524 1.524)) (justify right bottom))
+  (label "LED_1" (at 175.26 120.015 0)
+    (effects (font (size 1.524 1.524)) (justify left bottom))
+  )
+  (label "LED_2" (at 175.26 122.555 0)
+    (effects (font (size 1.524 1.524)) (justify left bottom))
+  )
+  (label "LED_3" (at 175.26 125.095 0)
+    (effects (font (size 1.524 1.524)) (justify left bottom))
   )
   (label "TIMEPULSE" (at 222.25 125.095 180)
     (effects (font (size 1.524 1.524)) (justify right bottom))
   )
-  (label "BTN" (at 232.41 28.575 0)
+  (label "TX1" (at 222.25 137.795 180)
+    (effects (font (size 1.524 1.524)) (justify right bottom))
+  )
+  (label "RX1" (at 222.25 140.335 180)
+    (effects (font (size 1.524 1.524)) (justify right bottom))
+  )
+  (label "BTN" (at 223.52 28.575 0)
     (effects (font (size 1.27 1.27)) (justify left bottom))
   )
@@
   (label "LED_3" (at 268.605 18.415 0)
     (effects (font (size 1.524 1.524)) (justify left bottom))
+  )
+  (global_label "PA0" (shape input) (at 175.26 38.735 0) (fields_autoplaced)
+    (effects (font (size 1.27 1.27)) (justify left))
+    (property "Intersheet References" "${INTERSHEET_REFS}" (id 0) (at 181.2412 38.6556 0)
+      (effects (font (size 1.27 1.27)) (justify left) hide)
+    )
+  )
+  (global_label "PA1" (shape input) (at 175.26 41.275 0) (fields_autoplaced)
+    (effects (font (size 1.27 1.27)) (justify left))
+    (property "Intersheet References" "${INTERSHEET_REFS}" (id 0) (at 181.2412 41.1956 0)
+      (effects (font (size 1.27 1.27)) (justify left) hide)
+    )
+  )
+  (global_label "COUNT_1_PCFO" (shape input) (at 175.26 88.265 0) (fields_autoplaced)
+    (effects (font (size 1.27 1.27)) (justify left))
+    (property "Intersheet References" "${INTERSHEET_REFS}" (id 0) (at 192.006 88.3444 0)
+      (effects (font (size 1.27 1.27)) (justify left) hide)
+    )
+  )
+  (global_label "COUNT_2" (shape input) (at 175.26 93.345 0) (fields_autoplaced)
+    (effects (font (size 1.27 1.27)) (justify left))
+    (property "Intersheet References" "${INTERSHEET_REFS}" (id 0) (at 186.0793 93.2656 0)
+      (effects (font (size 1.27 1.27)) (justify left) hide)
+    )
   )
   (symbol (lib_id "power:+3V3") (at 16.51 155.575 0) (unit 1)
@@
     (pin "1")
   )
+  (symbol (lib_id "power:GND") (at 223.52 41.275 0) (unit 1)
+    (in_bom yes) (on_board yes) (fields_autoplaced)
+    (property "Reference" "#PWR022" (id 0) (at 223.52 47.625 0)
+      (effects (font (size 1.27 1.27)) hide)
+    )
+    (property "Value" "GND" (id 1) (at 223.52 45.72 0))
+    (property "Footprint" "" (id 2) (at 223.52 41.275 0)
+      (effects (font (size 1.27 1.27)) hide)
+    )
+    (property "Datasheet" "" (id 3) (at 223.52 41.275 0)
+      (effects (font (size 1.27 1.27)) hide)
+    )
+    (pin "1")
+  )
   (symbol (lib_id "power:GND") (at 231.14 90.805 0) (unit 1)
     (in_bom yes) (on_board yes)
@@
     )
     (property "Datasheet" "" (id 3) (at 231.14 90.805 0)
-      (effects (font (size 1.27 1.27)) hide)
-    )
-    (pin "1")
-  )
-  (symbol (lib_id "power:GND") (at 232.41 41.275 0) (unit 1)
-    (in_bom yes) (on_board yes) (fields_autoplaced)
-    (property "Reference" "#PWR022" (id 0) (at 232.41 47.625 0)
-      (effects (font (size 1.27 1.27)) hide)
-    )
-    (property "Value" "GND" (id 1) (at 232.41 45.72 0))
-    (property "Footprint" "" (id 2) (at 232.41 41.275 0)
-      (effects (font (size 1.27 1.27)) hide)
-    )
-    (property "Datasheet" "" (id 3) (at 232.41 41.275 0)
       (effects (font (size 1.27 1.27)) hide)
     )
@@
     (pin "2")
   )
-  (symbol (lib_id "Switch:SW_Push") (at 232.41 33.655 90) (unit 1)
+  (symbol (lib_id "Switch:SW_Push") (at 223.52 33.655 90) (unit 1)
     (in_bom yes) (on_board yes) (fields_autoplaced)
-    (property "Reference" "SW1" (id 0) (at 233.68 32.3849 90)
+    (property "Reference" "SW1" (id 0) (at 224.79 32.3849 90)
       (effects (font (size 1.27 1.27)) (justify right))
     )
-    (property "Value" "SW_Push" (id 1) (at 233.68 34.9249 90)
+    (property "Value" "SW_Push" (id 1) (at 224.79 34.9249 90)
       (effects (font (size 1.27 1.27)) (justify right))
     )
-    (property "Footprint" "Button_Switch_SMD:SW_SPST_B3S-1000" (id 2) (at 227.33 33.655 0)
-      (effects (font (size 1.27 1.27)) hide)
-    )
-    (property "Datasheet" "~" (id 3) (at 227.33 33.655 0)
-      (effects (font (size 1.27 1.27)) hide)
-    )
+    (property "Footprint" "Button_Switch_SMD:SW_SPST_B3S-1000" (id 2) (at 218.44 33.655 0)
+      (effects (font (size 1.27 1.27)) hide)
+    )
+    (property "Datasheet" "~" (id 3) (at 218.44 33.655 0)
+      (effects (font (size 1.27 1.27)) hide)
+    )

Commit message: Edit shema and PCB
Parts:
- added JP?: SolderJumper_3_Bridged12, Jumper:SolderJumper-3_P1.3mm_Bridged12_RoundedPad1.0x1.5mm, symbol Jumper:SolderJumper_3_Bridged12
- added R19, R20: 100R, Resistor_SMD:R_0603_1608Metric, symbol SHT31V01A-rescue:R
- SW1: value SW_Push -> KMT031 NGJ LHS C&K; footprint Button_Switch_SMD:SW_SPST_B3S-1000 -> Mlab_SW:KMT031 NGJ LHS C&K
Connections:
- net +3V3: now also JP?.3 (B)
- net GND: now also JP?.1 (A); no longer U7.2 (ADDR)
- net PC0: now also R20.1
- net PC1: now also R19.1
- net EXTINT: now reaches J5.2
- net EXTINT: now also U8.40 ((PCINT8/T0/XCK)PB0)
- net GEO_STAT: now reaches J5.3
- net GEO_STAT: now also U8.41 ((PCINT9/CLKO/T1)PB1)
- net at J5.4: now also R19.2
- net at J5.5: now also R20.2
- new net: JP?.2 (C), U7.2 (ADDR)
- no-connect marks 23 -> 17
Other:
- note added: "Addres 0x58"
- note added: "Default addr 0x44"
- moved on the sheet: R12, R13, U7

Commit message: Edit schema
Connections:
- net COUNT_1_PCFO: now also U8.40 ((PCINT8/T0/XCK)PB0); no longer U8.21 ((PCINT18/TCK)PC2)
- net EXTINT: now also U8.42 ((PCINT10/AIN0/INT2)PB2); no longer U8.40 ((PCINT8/T0/XCK)PB0)
- net TIMEPULSE: now also U8.13 ((PCINT28/XCK1/OC1B)PD4); no longer U8.22 ((PCINT19/TMS)PC3)
Changed lines of the file:
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@@
   (no_connect (at 172.72 53.975))
   (no_connect (at 172.72 56.515))
-  (no_connect (at 172.72 66.675))
   (no_connect (at 172.72 69.215))
   (no_connect (at 172.72 71.755))
+  (no_connect (at 172.72 89.535))
+  (no_connect (at 172.72 92.075))
   (no_connect (at 172.72 99.695))
   (no_connect (at 172.72 102.235))
-  (no_connect (at 172.72 117.475))
   (no_connect (at 267.97 135.255))
   (no_connect (at 267.97 137.795))
@@
     (stroke (width 0) (type solid) (color 0 0 0 0))
   )
+  (wire (pts (xy 172.72 66.675) (xy 175.26 66.675))
+    (stroke (width 0) (type solid) (color 0 0 0 0))
+  )
   (wire (pts (xy 172.72 74.295) (xy 175.26 74.295))
     (stroke (width 0) (type solid) (color 0 0 0 0))
@@
     (stroke (width 0) (type solid) (color 0 0 0 0))
   )
-  (wire (pts (xy 172.72 89.535) (xy 175.26 89.535))
-    (stroke (width 0) (type solid) (color 0 0 0 0))
-  )
-  (wire (pts (xy 172.72 92.075) (xy 175.26 92.075))
-    (stroke (width 0) (type solid) (color 0 0 0 0))
-  )
   (wire (pts (xy 172.72 94.615) (xy 175.26 94.615))
     (stroke (width 0) (type solid) (color 0 0 0 0))
@@
     (stroke (width 0) (type solid) (color 0 0 0 0))
   )
+  (wire (pts (xy 172.72 117.475) (xy 175.26 117.475))
+    (stroke (width 0) (type solid) (color 0 0 0 0))
+  )
   (wire (pts (xy 172.72 120.015) (xy 175.26 120.015))
     (stroke (width 0) (type solid) (color 0 0 0 0))
@@
     (stroke (width 0) (type solid) (color 0 0 0 0))
   )
+  (wire (pts (xy 175.26 61.595) (xy 175.26 60.325))
+    (stroke (width 0) (type solid) (color 0 0 0 0))
+  )
   (wire (pts (xy 175.26 64.135) (xy 172.72 64.135))
-    (stroke (width 0) (type solid) (color 0 0 0 0))
-  )
-  (wire (pts (xy 175.26 88.265) (xy 175.26 89.535))
     (stroke (width 0) (type solid) (color 0 0 0 0))
   )
@@
     (effects (font (size 1.524 1.524)) (justify left bottom))
   )
-  (label "EXTINT" (at 175.26 61.595 0)
-    (effects (font (size 1.27 1.27)) (justify left bottom))
-  )
   (label "GEO_STAT" (at 175.26 64.135 0)
     (effects (font (size 1.27 1.27)) (justify left bottom))
   )
+  (label "EXTINT" (at 175.26 66.675 0)
+    (effects (font (size 1.27 1.27)) (justify left bottom))
+  )
   (label "PB5" (at 175.26 74.295 0)
     (effects (font (size 1.524 1.524)) (justify left bottom))
@@
   )
   (label "PC1" (at 175.26 86.995 0)
-    (effects (font (size 1.524 1.524)) (justify left bottom))
-  )
-  (label "TIMEPULSE" (at 175.26 92.075 0)
     (effects (font (size 1.524 1.524)) (justify left bottom))
   )
@@
   )
   (label "TX1" (at 175.26 114.935 0)
+    (effects (font (size 1.524 1.524)) (justify left bottom))
+  )
+  (label "TIMEPULSE" (at 175.26 117.475 0)
     (effects (font (size 1.524 1.524)) (justify left bottom))
   )
@@
     )
   )
-  (global_label "COUNT_1_PCFO" (shape input) (at 175.26 88.265 0) (fields_autoplaced)
+  (global_label "COUNT_1_PCFO" (shape input) (at 175.26 60.325 0) (fields_autoplaced)
     (effects (font (size 1.27 1.27)) (justify left))
-    (property "Intersheet References" "${INTERSHEET_REFS}" (id 0) (at 192.006 88.3444 0)
+    (property "Intersheet References" "${INTERSHEET_REFS}" (id 0) (at 192.006 60.4044 0)
       (effects (font (size 1.27 1.27)) (justify left) hide)
     )

Commit message: edit PCB
Parts:
- gave numbers to parts that had none: 1
Changed lines of the file:
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@@
   (symbol (lib_id "power:+3V3") (at 26.67 155.575 0) (unit 1)
     (in_bom yes) (on_board yes)
-    (property "Reference" "#PWR?" (id 0) (at 26.67 159.385 0)
+    (property "Reference" "#PWR0102" (id 0) (at 26.67 159.385 0)
       (effects (font (size 1.27 1.27)) hide)
     )
@@
   (symbol (lib_id "power:GND") (at 26.67 191.135 0) (unit 1)
     (in_bom yes) (on_board yes)
-    (property "Reference" "#PWR?" (id 0) (at 26.67 197.485 0)
+    (property "Reference" "#PWR0103" (id 0) (at 26.67 197.485 0)
       (effects (font (size 1.27 1.27)) hide)
     )
@@
   (symbol (lib_id "Jumper:SolderJumper_3_Bridged12") (at 26.67 180.975 90) (unit 1)
     (in_bom yes) (on_board yes)
-    (property "Reference" "JP?" (id 0) (at 25.019 179.8256 90)
-      (effects (font (size 1.27 1.27)) (justify left))
-    )
+    (property "Reference" "JP1" (id 0) (at 25.019 179.8256 90)
+      (effects (font (size 1.27 1.27)) (justify left))
+    )

Commit message: Edit PCB
Parts:
- removed JP1: SolderJumper_3_Bridged12, Jumper:SolderJumper-3_P1.3mm_Bridged12_RoundedPad1.0x1.5mm, symbol Jumper:SolderJumper_3_Bridged12
Connections:
- net GND: now also U7.2 (ADDR)
Changed lines of the file:
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@@
     (stroke (width 0) (type solid) (color 0 0 0 0))
   )
-  (wire (pts (xy 26.67 155.575) (xy 26.67 175.895))
-    (stroke (width 0) (type solid) (color 0 0 0 0))
-  )
-  (wire (pts (xy 26.67 186.055) (xy 26.67 191.135))
+  (wire (pts (xy 26.67 180.975) (xy 26.67 191.135))
+    (stroke (width 0) (type solid) (color 0 0 0 0))
+  )
+  (wire (pts (xy 26.67 180.975) (xy 31.115 180.975))
     (stroke (width 0) (type solid) (color 0 0 0 0))
   )
@@
   )
   (wire (pts (xy 29.21 31.115) (xy 29.21 29.845))
-    (stroke (width 0) (type solid) (color 0 0 0 0))
-  )
-  (wire (pts (xy 30.48 180.975) (xy 31.115 180.975))
     (stroke (width 0) (type solid) (color 0 0 0 0))
   )
@@
     (pin "1")
   )
-  (symbol (lib_id "power:+3V3") (at 26.67 155.575 0) (unit 1)
-    (in_bom yes) (on_board yes)
-    (property "Reference" "#PWR0102" (id 0) (at 26.67 159.385 0)
-      (effects (font (size 1.27 1.27)) hide)
-    )
-    (property "Value" "+3V3" (id 1) (at 27.051 151.1808 0))
-    (property "Footprint" "" (id 2) (at 26.67 155.575 0)
-      (effects (font (size 1.27 1.27)) hide)
-    )
-    (property "Datasheet" "" (id 3) (at 26.67 155.575 0)
-      (effects (font (size 1.27 1.27)) hide)
-    )
-    (pin "1")
-  )
   (symbol (lib_id "power:+3V3") (at 56.515 155.575 0) (unit 1)
     (in_bom yes) (on_board yes)
@@
     (pin "2")
   )
-  (symbol (lib_id "Jumper:SolderJumper_3_Bridged12") (at 26.67 180.975 90) (unit 1)
-    (in_bom yes) (on_board yes)
-    (property "Reference" "JP1" (id 0) (at 25.019 179.8256 90)
-      (effects (font (size 1.27 1.27)) (justify left))
-    )
-    (property "Value" "SolderJumper_3_Bridged12" (id 1) (at 25.019 182.1243 90)
-      (effects (font (size 1.27 1.27)) (justify left) hide)
-    )
-    (property "Footprint" "Jumper:SolderJumper-3_P1.3mm_Bridged12_RoundedPad1.0x1.5mm" (id 2) (at 26.67 180.975 0)
-      (effects (font (size 1.27 1.27)) hide)
-    )
-    (property "Datasheet" "~" (id 3) (at 26.67 180.975 0)
-      (effects (font (size 1.27 1.27)) hide)
-    )
-    (pin "1")
-    (pin "2")
-    (pin "3")
-  )
   (symbol (lib_id "Device:Crystal_GND24") (at 66.04 59.055 0) (unit 1)

Commit message: Edit PCB
Parts:
- added D6: RED, LED_SMD:LED_0603_1608Metric, symbol DATALOGGER01A-rescue:LED-device
- added R21: 2k2, Resistor_SMD:R_0603_1608Metric, symbol DATALOGGER01A-rescue:R-device
- C11, C12, C13, C14, C16, C18, C19, C20, C23, C24: UST_ID (none) -> 5c70984812875079b91f8bf2
- C21: UST_ID (none) -> 5c70984812875079b91f8bbe
- D3, D4, D5: UST_ID (none) -> 60d581db1287500165f859a2
- R12, R13, R14: UST_ID (none) -> 5c70984512875079b91f8962
- R15, R18, R5: UST_ID (none) -> 5c70984512875079b91f895e
- R16, R17: UST_ID (none) -> 5c70984512875079b91f8952
- R19, R20: UST_ID (none) -> 5c70984512875079b91f8956
- SW1: UST_ID (none) -> 612515a61287500165a9771d
- U7: UST_ID (none) -> 5c70984612875079b91f89e4
- Y1: UST_ID (none) -> 612516381287500165a97743
Connections:
- net +3V3: now also R21.2
- net GND: now also D6.1 (K)
- new net: D6.2 (A), R21.1
Other:
- moved on the sheet: SW1

Commit message: Edit PCB
Parts:
- C15, C17: value x pF -> 15 pF; UST_ID (none) -> 5c70984812875079b91f8be4
- D3: value RED -> YELLOW; UST_ID 60d581db1287500165f859a2 -> 60d582a31287500165f859f8
- D4: value RED -> BLUE; UST_ID 60d581db1287500165f859a2 -> 60d582f21287500165f85a23
- D5: value RED -> GREEN; UST_ID 60d581db1287500165f859a2 -> 60d582331287500165f859d0
Changed lines of the file:
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@@
-(kicad_sch (version 20210621) (generator eeschema)
+(kicad_sch (version 20210406) (generator eeschema)
   (paper "A4")
   (junction (at 17.78 20.955) (diameter 1.016) (color 0 0 0 0))
@@
       (effects (font (size 1.27 1.27)) (justify right))
     )
-    (property "Value" "RED" (id 1) (at 240.03 29.845 0)
+    (property "Value" "BLUE" (id 1) (at 240.03 29.845 0)
       (effects (font (size 1.27 1.27)) (justify right))
     )
@@
       (effects (font (size 1.27 1.27)) hide)
     )
-    (property "UST_ID" "60d581db1287500165f859a2" (id 5) (at 243.84 33.655 0)
+    (property "UST_ID" "60d582f21287500165f85a23" (id 5) (at 243.84 33.655 0)
       (effects (font (size 1.27 1.27)) hide)
     )
@@
       (effects (font (size 1.27 1.27)) (justify right))
     )
-    (property "Value" "RED" (id 1) (at 252.73 29.845 0)
+    (property "Value" "YELLOW" (id 1) (at 252.73 29.845 0)
       (effects (font (size 1.27 1.27)) (justify right))
     )
@@
       (effects (font (size 1.27 1.27)) hide)
     )
-    (property "UST_ID" "60d581db1287500165f859a2" (id 5) (at 256.54 33.655 0)
+    (property "UST_ID" "60d582a31287500165f859f8" (id 5) (at 256.54 33.655 0)
       (effects (font (size 1.27 1.27)) hide)
     )
@@
       (effects (font (size 1.27 1.27)) (justify right))
     )
-    (property "Value" "RED" (id 1) (at 264.795 29.845 0)
+    (property "Value" "GREEN" (id 1) (at 264.795 29.845 0)
       (effects (font (size 1.27 1.27)) (justify right))
     )
@@
       (effects (font (size 1.27 1.27)) hide)
     )
-    (property "UST_ID" "60d581db1287500165f859a2" (id 5) (at 268.605 33.655 0)
+    (property "UST_ID" "60d582331287500165f859d0" (id 5) (at 268.605 33.655 0)
       (effects (font (size 1.27 1.27)) hide)
     )
@@
       (effects (font (size 1.27 1.27)) (justify left))
     )
-    (property "Value" "x pF" (id 1) (at 51.181 67.818 0)
+    (property "Value" "15 pF" (id 1) (at 51.181 67.818 0)
       (effects (font (size 1.27 1.27)) (justify left))
     )
@@
       (effects (font (size 1.27 1.27)) hide)
     )
-    (property "UST_ID" "" (id 5) (at 59.69 66.675 0)
+    (property "UST_ID" "5c70984812875079b91f8be4" (id 5) (at 59.69 66.675 0)
       (effects (font (size 1.27 1.27)) hide)
     )
@@
       (effects (font (size 1.27 1.27)) (justify left))
     )
-    (property "Value" "x pF" (id 1) (at 77.851 67.818 0)
+    (property "Value" "15 pF" (id 1) (at 77.851 67.818 0)
       (effects (font (size 1.27 1.27)) (justify left))
     )
@@
       (effects (font (size 1.27 1.27)) hide)
     )
-    (property "UST_ID" "" (id 5) (at 74.93 66.675 0)
-      (effects (font (size 1.27 1.27)) hide)
-    )
+    (property "UST_ID" "5c70984812875079b91f8be4" (id 5) (at 74.93 66.675 0)
+      (effects (font (size 1.27 1.27)) hide)
+    )
