File: hw/sch_pcb/USTTHUNDERMILLPCB01A/USTTHUNDERMILLPCB01A.kicad_sch (KiCad schematic)
At the start: 11 parts, among them U1 ISL21080DIH312Z-TK 1V25, U2 OPA314

Commit message: Edit schema
Connections:
- net A0 renamed PA0
Other:
- added sheet CPU (CPU.kicad_sch)

Commit message: Edit
Parts:
- C1: UST_ID 5c70984712875079b91f8b4c -> (none)
- C2, C3, C4, C5, R1, R2, R3: footprint (none) -> Mlab_R:SMD-0805
Changed lines of the file:
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@@
       (effects (font (size 1.27 1.27)) (justify left))
     )
-    (property "Footprint" "" (id 2) (at 104.267 74.93 90)
+    (property "Footprint" "Mlab_R:SMD-0805" (id 2) (at 104.267 74.93 90)
       (effects (font (size 1.27 1.27)) hide)
     )
@@
       (effects (font (size 1.27 1.27)) (justify right))
     )
-    (property "Footprint" "" (id 2) (at 129.413 119.38 90)
+    (property "Footprint" "Mlab_R:SMD-0805" (id 2) (at 129.413 119.38 90)
       (effects (font (size 1.27 1.27)) hide)
     )
@@
     (property "Reference" "R3" (id 0) (at 137.795 104.1358 90))
     (property "Value" "10k" (id 1) (at 144.145 108.3395 90))
-    (property "Footprint" "" (id 2) (at 139.065 108.458 90)
+    (property "Footprint" "Mlab_R:SMD-0805" (id 2) (at 139.065 108.458 90)
       (effects (font (size 1.27 1.27)) hide)
     )
@@
       (effects (font (size 1.27 1.27)) hide)
     )
-    (property "UST_ID" "5c70984712875079b91f8b4c" (id 4) (at 36.83 34.29 0)
+    (property "UST_ID" "" (id 4) (at 36.83 34.29 0)
       (effects (font (size 1.27 1.27)) hide)
     )
@@
     (property "Reference" "C2" (id 0) (at 99.06 76.9578 90))
     (property "Value" "100nF" (id 1) (at 99.06 79.2565 90))
-    (property "Footprint" "" (id 2) (at 102.87 81.5848 0)
+    (property "Footprint" "Mlab_R:SMD-0805" (id 2) (at 102.87 81.5848 0)
       (effects (font (size 1.27 1.27)) hide)
     )
@@
       (effects (font (size 1.27 1.27)) (justify right))
     )
-    (property "Footprint" "" (id 2) (at 126.6698 125.73 0)
+    (property "Footprint" "Mlab_R:SMD-0805" (id 2) (at 126.6698 125.73 0)
       (effects (font (size 1.27 1.27)) hide)
     )
@@
     (property "Reference" "C4" (id 0) (at 137.795 109.9778 90))
     (property "Value" "1nF" (id 1) (at 139.065 117.9915 90))
-    (property "Footprint" "" (id 2) (at 142.875 112.6998 0)
+    (property "Footprint" "Mlab_R:SMD-0805" (id 2) (at 142.875 112.6998 0)
       (effects (font (size 1.27 1.27)) hide)
     )
@@
       (effects (font (size 1.27 1.27)) (justify right))
     )
-    (property "Footprint" "" (id 2) (at 143.1798 66.04 0)
+    (property "Footprint" "Mlab_R:SMD-0805" (id 2) (at 143.1798 66.04 0)
       (effects (font (size 1.27 1.27)) hide)
     )
@@
     )
     (path "/b83b274c-ccfa-487a-b887-d60edb6bc989"
-      (reference "C2") (unit 1) (value "100nF") (footprint "")
+      (reference "C2") (unit 1) (value "100nF") (footprint "Mlab_R:SMD-0805")
     )
     (path "/b2939f1c-82a1-477f-ab9e-8f0f059410cb"
-      (reference "C3") (unit 1) (value "100nF") (footprint "")
+      (reference "C3") (unit 1) (value "100nF") (footprint "Mlab_R:SMD-0805")
     )
     (path "/0f6f2db3-a7b7-477a-92e8-97cb6c9e5770"
-      (reference "C4") (unit 1) (value "1nF") (footprint "")
+      (reference "C4") (unit 1) (value "1nF") (footprint "Mlab_R:SMD-0805")
     )
     (path "/9eb0e1db-c7c4-42dc-b463-186a586dba42"
-      (reference "C5") (unit 1) (value "100nF") (footprint "")
+      (reference "C5") (unit 1) (value "100nF") (footprint "Mlab_R:SMD-0805")
     )
     (path "/cb25dd8d-ef4d-4bc3-bd88-f5c5fef4ca40"
@@
     )
     (path "/8095ce0f-c3fd-49f6-bf8f-97d0f7cadba6"
-      (reference "R1") (unit 1) (value "10M") (footprint "")
+      (reference "R1") (unit 1) (value "10M") (footprint "Mlab_R:SMD-0805")
     )
     (path "/4f9882c6-d303-4c4d-b24f-26b769c54bb2"
-      (reference "R2") (unit 1) (value "2k2") (footprint "")
+      (reference "R2") (unit 1) (value "2k2") (footprint "Mlab_R:SMD-0805")
     )
     (path "/446957a4-3a84-470b-98d5-90840b819a54"
-      (reference "R3") (unit 1) (value "10k") (footprint "")
+      (reference "R3") (unit 1) (value "10k") (footprint "Mlab_R:SMD-0805")
     )
     (path "/c1e857df-4d2d-4fe5-a2d4-b2f2f24786c5"
@@
     )
     (path "/c65d3f2e-8a0d-4ec9-900d-154ccfd9e32b/8eb7ea82-74a7-4824-94e8-99ca3ca20952"
-      (reference "D3") (unit 1) (value "Green 2mA") (footprint "")
+      (reference "D3") (unit 1) (value "Green 2mA") (footprint "LED_SMD:LED_0603_1608Metric")
     )
     (path "/c65d3f2e-8a0d-4ec9-900d-154ccfd9e32b/9714e962-7c24-4ce5-97e5-ab917ad32a0f"

Commit message: Edit PCB
Parts:
- C1, C2, C3, C4, C5: footprint Mlab_R:SMD-0805 -> Capacitor_SMD:C_0603_1608Metric
- D1: footprint (none) -> Diode_SMD:D_SMA
- R1, R2, R3: footprint Mlab_R:SMD-0805 -> Resistor_SMD:R_0603_1608Metric

Commit message: Edit PCB
Parts:
- D1: value 3v3 bipolární -> UCLAMP3301H.TCT; footprint Diode_SMD:D_SMA -> Diode_SMD:D_SOD-523
Changed lines of the file:
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@@
   )
   (symbol (lib_id "Diode:SD05_SOD323") (at 109.22 88.9 90) (unit 1)
-    (in_bom yes) (on_board yes) (fields_autoplaced)
+    (in_bom yes) (on_board yes)
     (property "Reference" "D1" (id 0) (at 111.2267 88.1391 90)
       (effects (font (size 1.27 1.27)) (justify right))
     )
-    (property "Value" "3v3 bipolární" (id 1) (at 111.2267 90.4378 90)
-      (effects (font (size 1.27 1.27)) (justify right))
-    )
-    (property "Footprint" "Diode_SMD:D_SMA" (id 2) (at 114.3 88.9 0)
-      (effects (font (size 1.27 1.27)) hide)
-    )
-    (property "Datasheet" "" (id 3) (at 109.22 88.9 0)
+    (property "Value" "UCLAMP3301H.TCT" (id 1) (at 105.5117 85.9928 0)
+      (effects (font (size 1.27 1.27)) (justify right))
+    )
+    (property "Footprint" "Diode_SMD:D_SOD-523" (id 2) (at 114.3 88.9 0)
+      (effects (font (size 1.27 1.27)) hide)
+    )
+    (property "Datasheet" "https://cz.mouser.com/datasheet/2/761/uclamp3301h-1278370.pdf" (id 3) (at 109.22 88.9 0)
       (effects (font (size 1.27 1.27)) hide)
     )
@@
     )
     (path "/cb25dd8d-ef4d-4bc3-bd88-f5c5fef4ca40"
-      (reference "D1") (unit 1) (value "3v3 bipolární") (footprint "Diode_SMD:D_SMA")
+      (reference "D1") (unit 1) (value "UCLAMP3301H.TCT") (footprint "Diode_SMD:D_SOD-523")
     )
     (path "/8095ce0f-c3fd-49f6-bf8f-97d0f7cadba6"
@@
       (reference "#PWR078") (unit 1) (value "GND") (footprint "")
     )
+    (path "/f1d72f98-8869-41cc-b10e-5c93f9725bfa/24529d8c-5e3f-4e94-aa1f-db1dcf48127f"
+      (reference "#PWR0101") (unit 1) (value "GND") (footprint "")
+    )
     (path "/f1d72f98-8869-41cc-b10e-5c93f9725bfa/0d7f9500-d88c-4d31-9b22-c38f725cd843"
       (reference "C11") (unit 1) (value "100nF") (footprint "Capacitor_SMD:C_0603_1608Metric")
@@
     )
     (path "/f1d72f98-8869-41cc-b10e-5c93f9725bfa/6af2c86a-d10b-40e7-bccf-8f3fb6b00ef2"
-      (reference "J4") (unit 1) (value "HEADER_2x03") (footprint "Mlab_Pin_Headers:Straight_2x03")
+      (reference "J4") (unit 1) (value "HEADER_2x03") (footprint "Mlab_Pin_Headers:SMD_2x03")
     )
     (path "/f1d72f98-8869-41cc-b10e-5c93f9725bfa/b51072d2-b9ea-421f-96d0-835547638d94"
@@
     )
     (path "/f1d72f98-8869-41cc-b10e-5c93f9725bfa/fefffef2-b902-4577-8ac1-b36192c7493b"
-      (reference "L1") (unit 1) (value "10uH - LQH32CN100K23L") (footprint "Mlab_R:SMD-1210")
+      (reference "L1") (unit 1) (value "10uH - LQH32CN100K23L") (footprint "Inductor_SMD:L_1210_3225Metric")
     )
     (path "/f1d72f98-8869-41cc-b10e-5c93f9725bfa/2759ee60-2d0c-4266-8094-7be37367714e"
@@
       (reference "U9") (unit 1) (value "AT24CS64-SSHM") (footprint "Package_SO:SOIC-8_3.9x4.9mm_P1.27mm")
     )
-    (path "/f1d72f98-8869-41cc-b10e-5c93f9725bfa/6f8d9541-2acb-4e85-bf83-e09e206e9dcf"
-      (reference "Y1") (unit 1) (value "16MHz") (footprint "Mlab_XTAL:Crystal_HC49-U_Vertical")
-    )
-  )
+    (path "/f1d72f98-8869-41cc-b10e-5c93f9725bfa/af4d7c80-fbbc-46ee-9099-d44a707b5e8a"
+      (reference "Y1") (unit 1) (value "16MHz") (footprint "Mlab_XTAL:Crystal SMD CFPX-180")
+    )
+  )

Commit message: Uprava PCB
Other:
- note added: "Umístit JST-GH konektor 3 pin"
