File: hw/sch_pcb/USTTHUNDERMILLPCB01A/USTTHUNDERMILLPCB01A.kicad_sch (KiCad schematic)
At the start: 11 parts, among them U1 ISL21080DIH312Z-TK 1V25, U2 OPA314

Commit message: Edit PCB
Parts:
- added J2: SM03B-GHS-TB, Connector_JST:JST_GH_SM03B-GHS-TB_1x03-1MP_P1.25mm_Horizontal, symbol MLAB_CONNECTORS_JST:SM03B-GHS-TB
Connections:
- net GND: now also J2.1, J2.3, J2.MP
- net PA0: now also J2.2
Other:
- note removed: "Umístit JST-GH konektor 3 pin"

Commit message: Edit shema and PCB
Parts:
- removed D1: UCLAMP3301H.TCT, Diode_SMD:D_SOD-523, symbol Diode:SD05_SOD323
- added D1: UCLAMP3301H.TCT, Diode_SMD:D_SOD-523, symbol Diode:SM6T12A
Connections:
- net GND: now also D1.2 (A2)
- net at C2.2, R1.2, U2.3 (+): now also D1.1 (A1)
- net REF_1V25 renamed PA1
Changed lines of the file:
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@@
     (stroke (width 0) (type solid) (color 0 0 0 0))
   )
-  (wire (pts (xy 149.86 85.09) (xy 160.655 85.09))
+  (wire (pts (xy 149.86 85.09) (xy 167.64 85.09))
     (stroke (width 0) (type solid) (color 0 0 0 0))
   )
@@
     (stroke (width 0) (type solid) (color 0 0 0 0))
   )
-  (wire (pts (xy 156.845 87.63) (xy 160.655 87.63))
-    (stroke (width 0) (type solid) (color 0 0 0 0))
-  )
-  (wire (pts (xy 156.845 91.44) (xy 156.845 87.63))
+  (wire (pts (xy 163.83 88.265) (xy 167.64 88.265))
     (stroke (width 0) (type solid) (color 0 0 0 0))
   )
@@
     (effects (font (size 1.524 1.524)) (justify right bottom))
   )
-  (global_label "PA0" (shape input) (at 160.655 85.09 0) (fields_autoplaced)
+  (label "REF_1V25" (at 163.83 88.265 180)
+    (effects (font (size 1.524 1.524)) (justify right bottom))
+  )
+  (global_label "PA0" (shape input) (at 167.64 85.09 0) (fields_autoplaced)
     (effects (font (size 1.27 1.27)) (justify left))
-    (property "Intersheet References" "${INTERSHEET_REFS}" (id 0) (at 166.6362 85.0106 0)
+    (property "Intersheet References" "${INTERSHEET_REFS}" (id 0) (at 173.6212 85.0106 0)
       (effects (font (size 1.27 1.27)) (justify left) hide)
     )
   )
-  (global_label "PA1" (shape input) (at 160.655 87.63 0) (fields_autoplaced)
+  (global_label "PA1" (shape input) (at 167.64 88.265 0) (fields_autoplaced)
     (effects (font (size 1.27 1.27)) (justify left))
-    (property "Intersheet References" "${INTERSHEET_REFS}" (id 0) (at 166.6362 87.5506 0)
+    (property "Intersheet References" "${INTERSHEET_REFS}" (id 0) (at 173.6212 88.1856 0)
       (effects (font (size 1.27 1.27)) (justify left) hide)
     )
@@
     (pin "1")
   )
-  (symbol (lib_id "power:GND") (at 156.845 91.44 0) (unit 1)
-    (in_bom yes) (on_board yes) (fields_autoplaced)
-    (property "Reference" "#PWR010" (id 0) (at 156.845 97.79 0)
-      (effects (font (size 1.27 1.27)) hide)
-    )
-    (property "Value" "GND" (id 1) (at 156.845 95.7644 0))
-    (property "Footprint" "" (id 2) (at 156.845 91.44 0)
-      (effects (font (size 1.27 1.27)) hide)
-    )
-    (property "Datasheet" "" (id 3) (at 156.845 91.44 0)
-      (effects (font (size 1.27 1.27)) hide)
-    )
-    (pin "1")
-  )
   (symbol (lib_id "power:GND") (at 219.075 91.44 0) (unit 1)
     (in_bom yes) (on_board yes) (fields_autoplaced)
@@
     (pin "2")
   )
-  (symbol (lib_id "Diode:SD05_SOD323") (at 109.22 88.9 90) (unit 1)
-    (in_bom yes) (on_board yes)
-    (property "Reference" "D1" (id 0) (at 111.2267 88.1391 90)
-      (effects (font (size 1.27 1.27)) (justify right))
-    )
-    (property "Value" "UCLAMP3301H.TCT" (id 1) (at 105.5117 85.9928 0)
-      (effects (font (size 1.27 1.27)) (justify right))
-    )
-    (property "Footprint" "Diode_SMD:D_SOD-523" (id 2) (at 114.3 88.9 0)
-      (effects (font (size 1.27 1.27)) hide)
-    )
-    (property "Datasheet" "https://cz.mouser.com/datasheet/2/761/uclamp3301h-1278370.pdf" (id 3) (at 109.22 88.9 0)
+  (symbol (lib_id "Diode:SM6T12A") (at 109.22 88.9 270) (unit 1)
+    (in_bom yes) (on_board yes)
+    (property "Reference" "D1" (id 0) (at 111.2521 88.1391 90)
+      (effects (font (size 1.27 1.27)) (justify left))
+    )
+    (property "Value" "UCLAMP3301H.TCT" (id 1) (at 105.5371 85.9928 0)
+      (effects (font (size 1.27 1.27)) (justify left))
+    )
+    (property "Footprint" "Diode_SMD:D_SOD-523" (id 2) (at 104.14 88.9 0)
+      (effects (font (size 1.27 1.27)) hide)
+    )
+    (property "Datasheet" "https://www.st.com/resource/en/datasheet/sm6t.pdf" (id 3) (at 109.22 87.63 0)
       (effects (font (size 1.27 1.27)) hide)
     )
@@
       (reference "#PWR09") (unit 1) (value "GND") (footprint "")
     )
-    (path "/1117e817-1baa-41cc-90ca-20a5efcf81bf"
-      (reference "#PWR010") (unit 1) (value "GND") (footprint "")
-    )
     (path "/f70c077c-72e8-4340-be0a-fbb1a6a66741"
       (reference "#PWR020") (unit 1) (value "GND") (footprint "")
@@
       (reference "C5") (unit 1) (value "100nF") (footprint "Capacitor_SMD:C_0603_1608Metric")
     )
-    (path "/cb25dd8d-ef4d-4bc3-bd88-f5c5fef4ca40"
+    (path "/63710ae2-0173-429f-930e-1f82ffa3907c"
       (reference "D1") (unit 1) (value "UCLAMP3301H.TCT") (footprint "Diode_SMD:D_SOD-523")
     )
@@
       (reference "#PWR044") (unit 1) (value "GND") (footprint "")
     )
-    (path "/f1d72f98-8869-41cc-b10e-5c93f9725bfa/e0fd8af8-46c5-4b4c-916d-03fecee3d785"
-      (reference "#PWR045") (unit 1) (value "GND") (footprint "")
-    )
     (path "/f1d72f98-8869-41cc-b10e-5c93f9725bfa/33c3a7d2-ad6c-4221-9117-3fbba9d32dc4"
       (reference "#PWR046") (unit 1) (value "GND") (footprint "")
@@
       (reference "#PWR0101") (unit 1) (value "GND") (footprint "")
     )
+    (path "/f1d72f98-8869-41cc-b10e-5c93f9725bfa/15d4db8b-2807-4d91-b861-47ee9ffddfbd"
+      (reference "#PWR?") (unit 1) (value "GND") (footprint "")
+    )
+    (path "/f1d72f98-8869-41cc-b10e-5c93f9725bfa/9bb7bfdd-1666-4df1-8ac2-c499cbfd3ab8"
+      (reference "#PWR?") (unit 1) (value "+3V3") (footprint "")
+    )
     (path "/f1d72f98-8869-41cc-b10e-5c93f9725bfa/0d7f9500-d88c-4d31-9b22-c38f725cd843"
       (reference "C11") (unit 1) (value "100nF") (footprint "Capacitor_SMD:C_0603_1608Metric")
@@
       (reference "J6") (unit 1) (value "SM06B-GHS-TB") (footprint "Connector_JST:JST_GH_SM06B-GHS-TB_1x06-1MP_P1.25mm_Horizontal")
     )
+    (path "/f1d72f98-8869-41cc-b10e-5c93f9725bfa/0cde32ab-061f-4ecc-bf6c-d7b9c47305b4"
+      (reference "JP?") (unit 1) (value "SolderJumper_3_Bridged12") (footprint "Jumper:SolderJumper-3_P1.3mm_Bridged12_RoundedPad1.0x1.5mm")
+    )
     (path "/f1d72f98-8869-41cc-b10e-5c93f9725bfa/fefffef2-b902-4577-8ac1-b36192c7493b"
       (reference "L1") (unit 1) (value "10uH - LQH32CN100K23L") (footprint "Inductor_SMD:L_1210_3225Metric")
@@
       (reference "R18") (unit 1) (value "2k2") (footprint "Resistor_SMD:R_0603_1608Metric")
     )
+    (path "/f1d72f98-8869-41cc-b10e-5c93f9725bfa/447c6b1c-d0b8-4d04-9ac9-baf09bd2c7f1"
+      (reference "R19") (unit 1) (value "100R") (footprint "Resistor_SMD:R_0603_1608Metric")
+    )
+    (path "/f1d72f98-8869-41cc-b10e-5c93f9725bfa/715e05f2-19f2-4635-b5ac-c1a03b8ac678"
+      (reference "R20") (unit 1) (value "100R") (footprint "Resistor_SMD:R_0603_1608Metric")
+    )
     (path "/f1d72f98-8869-41cc-b10e-5c93f9725bfa/a4fcada3-4f52-46a5-ac5b-6f841abab351"
-      (reference "SW1") (unit 1) (value "SW_Push") (footprint "Button_Switch_SMD:SW_SPST_B3S-1000")
+      (reference "SW1") (unit 1) (value "KMT031 NGJ LHS C&K") (footprint "Mlab_SW:KMT031 NGJ LHS C&K")
     )
     (path "/f1d72f98-8869-41cc-b10e-5c93f9725bfa/a8a58eb8-010e-4d62-89ce-82d3f52d9321"

Commit message: Edit PCB
Changed lines of the file:
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@@
     (effects (font (size 1.524 1.524)) (justify left bottom))
-  )
-  (label "STATOR" (at 85.09 82.55 180)
-    (effects (font (size 1.27 1.27)) (justify right bottom))
-  )
-  (label "ROTOR_GND" (at 85.09 88.265 180)
-    (effects (font (size 1.27 1.27)) (justify right bottom))
   )
   (label "REF_1V25" (at 106.045 69.215 180)
@@
   (label "REF_1V25" (at 163.83 88.265 180)
     (effects (font (size 1.524 1.524)) (justify right bottom))
+  )
+  (global_label "STATOR" (shape input) (at 85.09 82.55 180) (fields_autoplaced)
+    (effects (font (size 1.27 1.27)) (justify right))
+    (property "Intersheet References" "${INTERSHEET_REFS}" (id 0) (at 75.8431 82.4706 0)
+      (effects (font (size 1.27 1.27)) (justify right) hide)
+    )
+  )
+  (global_label "ROTOR_GND" (shape input) (at 85.09 88.265 180) (fields_autoplaced)
+    (effects (font (size 1.27 1.27)) (justify right))
+    (property "Intersheet References" "${INTERSHEET_REFS}" (id 0) (at 71.6702 88.1856 0)
+      (effects (font (size 1.27 1.27)) (justify right) hide)
+    )
   )
   (global_label "PA0" (shape input) (at 167.64 85.09 0) (fields_autoplaced)
@@
       (reference "#PWR0101") (unit 1) (value "GND") (footprint "")
     )
-    (path "/f1d72f98-8869-41cc-b10e-5c93f9725bfa/9bb7bfdd-1666-4df1-8ac2-c499cbfd3ab8"
-      (reference "#PWR0102") (unit 1) (value "+3V3") (footprint "")
-    )
     (path "/f1d72f98-8869-41cc-b10e-5c93f9725bfa/15d4db8b-2807-4d91-b861-47ee9ffddfbd"
       (reference "#PWR0103") (unit 1) (value "GND") (footprint "")
@@
       (reference "J6") (unit 1) (value "SM06B-GHS-TB") (footprint "Connector_JST:JST_GH_SM06B-GHS-TB_1x06-1MP_P1.25mm_Horizontal")
     )
-    (path "/f1d72f98-8869-41cc-b10e-5c93f9725bfa/0cde32ab-061f-4ecc-bf6c-d7b9c47305b4"
-      (reference "JP1") (unit 1) (value "SolderJumper_3_Bridged12") (footprint "Jumper:SolderJumper-3_P1.3mm_Bridged12_RoundedPad1.0x1.5mm")
-    )
     (path "/f1d72f98-8869-41cc-b10e-5c93f9725bfa/fefffef2-b902-4577-8ac1-b36192c7493b"

Commit message: Edit PCB
Parts:
- C1, C2, C3, C5: UST_ID (none) -> 5c70984812875079b91f8bf2
- C4: UST_ID (none) -> 5c70984812875079b91f8bec
- D1: UST_ID (none) -> 612514fe1287500165a976f3
- R1: UST_ID (none) -> 5c70984712875079b91f8b6d
- R2: UST_ID (none) -> 5c70984512875079b91f895e
- R3: UST_ID (none) -> 5c70984512875079b91f8962
- U2: UST_ID (none) -> 5c70984412875079b91f879a
Changed lines of the file:
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@@
+      (effects (font (size 1.27 1.27)) hide)
+    )
+    (property "UST_ID" "5c70984712875079b91f8b6d" (id 4) (at 106.045 74.93 0)
       (effects (font (size 1.27 1.27)) hide)
     )
@@
     )
     (property "Datasheet" "~" (id 3) (at 127.635 119.38 0)
+      (effects (font (size 1.27 1.27)) hide)
+    )
+    (property "UST_ID" "5c70984512875079b91f895e" (id 4) (at 127.635 119.38 0)
       (effects (font (size 1.27 1.27)) hide)
     )
@@
       (effects (font (size 1.27 1.27)) hide)
     )
+    (property "UST_ID" "5c70984512875079b91f8962" (id 4) (at 139.065 106.68 0)
+      (effects (font (size 1.27 1.27)) hide)
+    )
     (pin "1")
     (pin "2")
@@
       (effects (font (size 1.27 1.27)) hide)
     )
+    (property "UST_ID" "612514fe1287500165a976f3" (id 4) (at 109.22 88.9 0)
+      (effects (font (size 1.27 1.27)) hide)
+    )
     (pin "1")
     (pin "2")
@@
       (effects (font (size 1.27 1.27)) hide)
     )
-    (property "UST_ID" "" (id 4) (at 36.83 34.29 0)
+    (property "UST_ID" "5c70984812875079b91f8bf2" (id 4) (at 36.83 34.29 0)
       (effects (font (size 1.27 1.27)) hide)
     )
@@
       (effects (font (size 1.27 1.27)) hide)
     )
+    (property "UST_ID" "5c70984812875079b91f8bf2" (id 4) (at 99.06 82.55 0)
+      (effects (font (size 1.27 1.27)) hide)
+    )
     (pin "1")
     (pin "2")
@@
     )
     (property "Datasheet" "~" (id 3) (at 127.635 129.54 0)
+      (effects (font (size 1.27 1.27)) hide)
+    )
+    (property "UST_ID" "5c70984812875079b91f8bf2" (id 4) (at 127.635 129.54 0)
       (effects (font (size 1.27 1.27)) hide)
     )
@@
       (effects (font (size 1.27 1.27)) hide)
     )
+    (property "UST_ID" "5c70984812875079b91f8bec" (id 4) (at 139.065 113.665 0)
+      (effects (font (size 1.27 1.27)) hide)
+    )
     (pin "1")
     (pin "2")
@@
     )
     (property "Datasheet" "~" (id 3) (at 144.145 69.85 0)
+      (effects (font (size 1.27 1.27)) hide)
+    )
+    (property "UST_ID" "5c70984812875079b91f8bf2" (id 4) (at 144.145 69.85 0)
       (effects (font (size 1.27 1.27)) hide)
     )
@@
     )
     (property "Datasheet" "https://www.ti.com/lit/ds/symlink/opa314-q1.pdf?HQS=dis-mous-null-mousermode-dsf-pf-null-wwe&ts=1627026622034&ref_url=https%253A%252F%252Fcz.mouser.com%252F" (id 3) (at 140.97 80.01 0)
+      (effects (font (size 1.27 1.27)) hide)
+    )
+    (property "UST_ID" "5c70984412875079b91f879a" (id 4) (at 140.97 85.09 0)
       (effects (font (size 1.27 1.27)) hide)
     )
@@
       (reference "#PWR0101") (unit 1) (value "GND") (footprint "")
     )
+    (path "/f1d72f98-8869-41cc-b10e-5c93f9725bfa/facbc6fd-2f6a-4de8-aa2c-cb33e3a11235"
+      (reference "#PWR0102") (unit 1) (value "+3V3") (footprint "")
+    )
     (path "/f1d72f98-8869-41cc-b10e-5c93f9725bfa/15d4db8b-2807-4d91-b861-47ee9ffddfbd"
       (reference "#PWR0103") (unit 1) (value "GND") (footprint "")
     )
+    (path "/f1d72f98-8869-41cc-b10e-5c93f9725bfa/50c7126d-1b29-4f77-8a94-a8a3731152fb"
+      (reference "#PWR0106") (unit 1) (value "GND") (footprint "")
+    )
     (path "/f1d72f98-8869-41cc-b10e-5c93f9725bfa/0d7f9500-d88c-4d31-9b22-c38f725cd843"
       (reference "C11") (unit 1) (value "100nF") (footprint "Capacitor_SMD:C_0603_1608Metric")
@@
       (reference "D5") (unit 1) (value "RED") (footprint "LED_SMD:LED_0603_1608Metric")
     )
+    (path "/f1d72f98-8869-41cc-b10e-5c93f9725bfa/a5056612-6744-4532-b64b-95fd1a6f9437"
+      (reference "D6") (unit 1) (value "RED") (footprint "LED_SMD:LED_0603_1608Metric")
+    )
     (path "/f1d72f98-8869-41cc-b10e-5c93f9725bfa/6af2c86a-d10b-40e7-bccf-8f3fb6b00ef2"
       (reference "J4") (unit 1) (value "HEADER_2x03") (footprint "Mlab_Pin_Headers:SMD_2x03")
@@
       (reference "R20") (unit 1) (value "100R") (footprint "Resistor_SMD:R_0603_1608Metric")
     )
+    (path "/f1d72f98-8869-41cc-b10e-5c93f9725bfa/e4198e5e-c89f-477e-946e-4262b67dcb4d"
+      (reference "R21") (unit 1) (value "2k2") (footprint "Resistor_SMD:R_0603_1608Metric")
+    )
     (path "/f1d72f98-8869-41cc-b10e-5c93f9725bfa/a4fcada3-4f52-46a5-ac5b-6f841abab351"
