File: hw/sch_pcb/USTTHUNDERMILLPCB01A/USTTHUNDERMILLPCB01A.kicad_sch (KiCad schematic)
At the start: 12 parts, among them J2 SM03B-GHS-TB, U1 ISL21080DIH312Z-TK 1V25, U2 OPA314

Commit message: Edit BOM
Parts:
- J2: UST_ID (none) -> 612880e51287500165a978de
Changed lines of the file:
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@@
       (effects (font (size 1.524 1.524)))
+    )
+    (property "UST_ID" "612880e51287500165a978de" (id 4) (at 227.33 85.09 0)
+      (effects (font (size 1.27 1.27)) hide)
     )
     (pin "1")
