File: hw/sch_pcb/USTTHUNDERMILLPCB01A/USTTHUNDERMILLPCB01A.kicad_pcb (KiCad board)
At the start: 2 copper layers, 80 x 80 mm, 59 parts, among them J1 SM04B-GHS-TB, J4 HEADER_2x03, J5 SM08B-GHS-TB, J6 SM06B-GHS-TB, U1 ISL21080DIH312Z-TK 1V25, U2 OPA314, U3 MIC5504-3.3YM5, U4 PCF8583, U5 VCNT2020, U6 VCNT2020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

Commit message: Edit PCB
Parts:
- moved C1 148.7 mm to (96.0, 90.2), turned to 90 degrees
- moved U1 138.1 mm to (92.9, 89.4)
- moved C21 92.6 mm to (159.7, 83.0), turned to 0 degrees
- moved C23 89.8 mm to (159.6, 85.5), turned to 0 degrees
- moved C24 72.9 mm to (151.9, 111.7), turned to 180 degrees
- moved C19 62.0 mm to (151.9, 96.9)
- moved C20 60.1 mm to (160.8, 101.1), turned to 0 degrees
- moved C18 46.3 mm to (168.3, 94.4)
- moved U7 44.8 mm to (144.6, 102.9)
- moved D4 38.2 mm to (162.9, 81.8)
- moved C16 37.6 mm to (163.8, 84.9)
- moved L1 32.4 mm to (167.6, 84.1), turned to 180 degrees
- moved R15 29.6 mm to (163.3, 80.1)
- moved C14 29.4 mm to (170.8, 85.4)
- moved Y1 29.0 mm to (161.1, 103.4)
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
Commit message: uprava PCB
Parts:
- added D5: RED, LED_SMD:LED_0603_1608Metric, F.Cu at (102.1, 62.7)
- added R18: 2k2, Resistor_SMD:R_0603_1608Metric, F.Cu at (102.1, 70.3)
- added SW1: SW_Push, Button_Switch_SMD:SW_SPST_B3S-1000, F.Cu at (94.5, 65.6)
- C15, C17: value 100nF -> x pF
- D3: value Green 2mA -> RED
- R5: value ? -> 2k2
- moved D3 68.5 mm to (102.1, 65.3), turned to 0 degrees
- moved R5 51.1 mm to (102.1, 67.8), turned to 0 degrees
Connections:
- D3 pad 1: Net-(D3-Pad1) -> GND
- D3 pad 2: GND -> Net-(D3-Pad2)
- J5 pad 6: (no net) -> /CPU/TX1
- J5 pad 7: (no net) -> /CPU/RX1
- R15 pad 2: /CPU/LED -> (no net)
- R5 pad 1: Net-(D3-Pad1) -> Net-(D3-Pad2)
- R5 pad 2: Net-(R5-Pad2) -> /CPU/LED_2
- U4 pad 2: Net-(R5-Pad2) -> (no net)
- U8 pad 11: (no net) -> /CPU/RX1
- U8 pad 12: (no net) -> /CPU/TX1
- U8 pad 26: /CPU/LED -> (no net)

Commit message: Edit PCB
Parts:
- added J2: SM03B-GHS-TB, Connector_JST:JST_GH_SM03B-GHS-TB_1x03-1MP_P1.25mm_Horizontal, F.Cu at (167.0, 139.1)
Connections:
- C1 pad 2: GND -> PA1
- C10 pad 2: GND -> PA1
- C11 pad 2: GND -> PA1
- C12 pad 2: GND -> PA1
- C13 pad 2: GND -> PA1
- C14 pad 2: GND -> PA1
- C15 pad 2: GND -> PA1
- C16 pad 2: GND -> PA1
- C17 pad 2: GND -> PA1
- C18 pad 2: GND -> PA1
- C19 pad 2: GND -> PA1
- C2 pad 1: (no net) -> /STATOR
- C20 pad 2: GND -> PA1
- C21 pad 2: GND -> PA1
- C23 pad 2: GND -> PA1
- C24 pad 2: GND -> PA1
- C3 pad 1: GND -> PA1
- C4 pad 2: /PA0 -> PA0
- C5 pad 1: GND -> PA1
- C6 pad 2: GND -> PA1
- C7 pad 2: GND -> PA1
- C8 pad 2: GND -> PA1
- C9 pad 2: GND -> PA1
- D1 pad 1: GND -> PA1
- D2 pad 2: GND -> PA1
- D3 pad 1: GND -> PA1
- D4 pad 1: GND -> PA1
- D5 pad 1: GND -> PA1
- J1 pad 4: GND -> PA1
- J1 pad MP: GND -> PA1
- J4 pad 6: GND -> PA1
- J5 pad 2: (no net) -> unconnected-(J5-Pad2)
- J5 pad 3: (no net) -> unconnected-(J5-Pad3)
- J5 pad 4: (no net) -> unconnected-(J5-Pad4)
- J5 pad 5: (no net) -> unconnected-(J5-Pad5)
- J5 pad 8: GND -> PA1
- J5 pad MP: GND -> PA1
- J6 pad 4: (no net) -> unconnected-(J6-Pad4)
- J6 pad 5: (no net) -> unconnected-(J6-Pad5)
- J6 pad 6: GND -> PA1
- J6 pad MP: GND -> PA1
- R11 pad 2: /tachometer/COUNT_2 -> COUNT_2
- R15 pad 2: (no net) -> /CPU/LED_1
- R3 pad 2: /PA0 -> PA0
- SW1 pad 1: GND -> PA1
- U1 pad 3: GND -> PA1
- U2 pad 1: /PA0 -> PA0
- U2 pad 2: GND -> PA1
- U3 pad 2: GND -> PA1
- U3 pad 4: (no net) -> unconnected-(U3-Pad4)
- U4 pad 2: (no net) -> COUNT_1_PCFO
- U4 pad 3: GND -> PA1
- U4 pad 4: GND -> PA1
- U4 pad 7: (no net) -> unconnected-(U4-Pad7)
- U5 pad 1: GND -> PA1
- U5 pad 4: GND -> PA1
- U6 pad 1: GND -> PA1
- U6 pad 2: /tachometer/COUNT_2 -> COUNT_2
- U6 pad 4: GND -> PA1
- U7 pad 2: GND -> PA1
- U7 pad 3: (no net) -> unconnected-(U7-Pad3)
- U7 pad 6: (no net) -> unconnected-(U7-Pad6)
- U7 pad 7: GND -> PA1
- U7 pad 8: GND -> PA1
- U7 pad 9: GND -> PA1
- U8 pad 13: (no net) -> unconnected-(U8-Pad13)
- U8 pad 14: (no net) -> /CPU/LED_1
- U8 pad 15: (no net) -> /CPU/LED_2
- U8 pad 16: (no net) -> /CPU/LED_3
- U8 pad 18: GND -> PA1
- U8 pad 21: (no net) -> COUNT_1_PCFO
- U8 pad 23: (no net) -> COUNT_2
- U8 pad 24: (no net) -> /CPU/BTN
- U8 pad 25: (no net) -> unconnected-(U8-Pad25)
- U8 pad 26: (no net) -> unconnected-(U8-Pad26)
- U8 pad 28: GND -> PA1
- U8 pad 30: (no net) -> unconnected-(U8-Pad30)
- U8 pad 31: (no net) -> unconnected-(U8-Pad31)
- U8 pad 32: (no net) -> unconnected-(U8-Pad32)
- U8 pad 33: (no net) -> unconnected-(U8-Pad33)
- U8 pad 34: (no net) -> unconnected-(U8-Pad34)
- U8 pad 35: (no net) -> unconnected-(U8-Pad35)
- U8 pad 36: (no net) -> PA1
- U8 pad 37: (no net) -> PA0
- U8 pad 39: GND -> PA1
- U8 pad 40: (no net) -> unconnected-(U8-Pad40)
- U8 pad 41: (no net) -> unconnected-(U8-Pad41)
- U8 pad 42: (no net) -> unconnected-(U8-Pad42)
- U8 pad 43: (no net) -> unconnected-(U8-Pad43)
- U8 pad 44: (no net) -> unconnected-(U8-Pad44)
- U8 pad 6: GND -> PA1
- U9 pad 1: GND -> PA1
- U9 pad 2: GND -> PA1
- U9 pad 3: GND -> PA1
- U9 pad 4: GND -> PA1
- U9 pad 7: GND -> PA1
- Y1 pad 2: GND -> PA1
- Y1 pad 4: GND -> PA1
Routing:
- net COUNT_2: track 0.00 -> 2.73 mm, vias 0 -> 1
- net /tachometer/COUNT_2: track 2.73 -> 0.00 mm, vias 1 -> 0
- net PA1: vias 0 -> 25
- net GND: vias 25 -> 0
- added copper zone on B.Cu, net PA1
- added copper zone on F.Cu, net PA1
- removed copper zone on B.Cu, net GND
- removed copper zone on F.Cu, net GND

Commit message: Edit shema and PCB
Parts:
- added R19: 100R, Resistor_SMD:R_0603_1608Metric, F.Cu at (111.8, 92.7)
- added R20: 100R, Resistor_SMD:R_0603_1608Metric, F.Cu at (111.8, 94.5)
- SW1: value SW_Push -> KMT031 NGJ LHS C&K; footprint Button_Switch_SMD:SW_SPST_B3S-1000 -> Mlab_SW:KMT031 NGJ LHS C&K
- moved C10 84.0 mm to (137.3, 60.0)
- moved C9 83.2 mm to (134.7, 59.9)
- moved J2 82.8 mm to (107.7, 81.3), turned to -108 degrees
- moved D3 82.3 mm to (178.8, 95.0), turned to 180 degrees
- moved D5 82.1 mm to (178.8, 92.0), turned to 180 degrees
- moved R4 81.8 mm to (131.7, 60.5), turned to 180 degrees
- moved C8 81.1 mm to (127.5, 61.0), turned to 0 degrees
- moved U3 78.5 mm to (127.5, 64.3), turned to 90 degrees
- moved R5 78.1 mm to (175.3, 95.0), turned to 180 degrees
- moved C7 77.7 mm to (124.0, 65.5), turned to 135 degrees
- moved D2 77.6 mm to (119.4, 68.5), turned to 135 degrees
- moved C6 77.0 mm to (122.1, 67.1), turned to 135 degrees
- moved SW1 76.5 mm to (170.4, 75.3)
- moved R18 76.4 mm to (175.3, 92.0), turned to 180 degrees
- moved J5 72.0 mm to (106.6, 94.1), turned to -87 degrees
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Connections:
- C1 pad 1: /REF_1V25 -> PA1
- C1 pad 2: PA1 -> (no net)
- C10 pad 2: PA1 -> (no net)
- C11 pad 2: PA1 -> (no net)
- C12 pad 2: PA1 -> (no net)
- C13 pad 2: PA1 -> (no net)
- C14 pad 2: PA1 -> (no net)
- C15 pad 2: PA1 -> (no net)
- C16 pad 2: PA1 -> (no net)
- C17 pad 2: PA1 -> (no net)
- C18 pad 2: PA1 -> (no net)
- C19 pad 2: PA1 -> (no net)
- C20 pad 2: PA1 -> (no net)
- C21 pad 2: PA1 -> (no net)
- C23 pad 2: PA1 -> (no net)
- C24 pad 2: PA1 -> (no net)
- C3 pad 1: PA1 -> (no net)
- C3 pad 2: /REF_1V25 -> PA1
- C5 pad 1: PA1 -> (no net)
- C6 pad 2: PA1 -> (no net)
- C7 pad 2: PA1 -> (no net)
- C8 pad 2: PA1 -> (no net)
- C9 pad 2: PA1 -> (no net)
- D1 pad 1: PA1 -> Net-(C2-Pad2)
- D1 pad 2: Net-(C2-Pad2) -> (no net)
- D2 pad 2: PA1 -> (no net)
- D3 pad 1: PA1 -> (no net)
- D4 pad 1: PA1 -> (no net)
- D5 pad 1: PA1 -> (no net)
- J1 pad 4: PA1 -> (no net)
- J1 pad MP: PA1 -> (no net)
- J2 pad 1: PA1 -> (no net)
- J2 pad 3: PA1 -> (no net)
- J2 pad MP: PA1 -> (no net)
- J4 pad 6: PA1 -> (no net)
- J5 pad 2: unconnected-(J5-Pad2) -> /CPU/EXTINT
- J5 pad 3: unconnected-(J5-Pad3) -> /CPU/GEO_STAT
- J5 pad 4: unconnected-(J5-Pad4) -> Net-(J5-Pad4)
- J5 pad 5: unconnected-(J5-Pad5) -> Net-(J5-Pad5)
- J5 pad 8: PA1 -> (no net)
- J5 pad MP: PA1 -> (no net)
- J6 pad 6: PA1 -> (no net)
- J6 pad MP: PA1 -> (no net)
- R1 pad 1: /REF_1V25 -> PA1
- R2 pad 1: /REF_1V25 -> PA1
- SW1 pad 1: PA1 -> (no net)
- U1 pad 2: /REF_1V25 -> PA1
- U1 pad 3: PA1 -> (no net)
- U2 pad 2: PA1 -> (no net)
- U3 pad 2: PA1 -> (no net)
- U4 pad 3: PA1 -> (no net)
- U4 pad 4: PA1 -> (no net)
- U5 pad 1: PA1 -> (no net)
- U5 pad 4: PA1 -> (no net)
- U6 pad 1: PA1 -> (no net)
- U6 pad 4: PA1 -> (no net)
- U7 pad 2: PA1 -> (no net)
- U7 pad 7: PA1 -> (no net)
- U7 pad 8: PA1 -> (no net)
- U7 pad 9: PA1 -> (no net)
- U8 pad 18: PA1 -> (no net)
- U8 pad 28: PA1 -> (no net)
- U8 pad 39: PA1 -> (no net)
- U8 pad 40: unconnected-(U8-Pad40) -> /CPU/EXTINT
- U8 pad 41: unconnected-(U8-Pad41) -> /CPU/GEO_STAT
- U8 pad 6: PA1 -> (no net)
- U9 pad 1: PA1 -> (no net)
- U9 pad 2: PA1 -> (no net)
- U9 pad 3: PA1 -> (no net)
- U9 pad 4: PA1 -> (no net)
- U9 pad 7: PA1 -> (no net)
- Y1 pad 2: PA1 -> (no net)
- Y1 pad 4: PA1 -> (no net)
Routing:
- net PA1: vias 25 -> 21
Other:
- copper layers 2 -> 4
