File: hw/sch_pcb/USTTHUNDERMILLPCB01A/tachometer.kicad_sch (KiCad schematic)
At the start: 38 parts, among them J1 SM04B-GHS-TB, J2 SM04B-GHS-TB, U3 SN74LVC1G14-Q1, U4 MIC5504-3.3YM5, U5 SN74LVC1G14-Q1, U6 PCF8583, U7 VCNT2020, U8 VCNT2020

Commit message: Edit schema
Parts:
- removed C10, C11, C19, C20, C9: 100nF, Mlab_R:SMD-0603, symbol Device:C
- removed C13: 47uF, Mlab_C:TantalC_SizeC_Reflow, symbol SPACEDOS01A_PCB01A-rescue:CP-Device
- removed C14: 10uF, Mlab_R:SMD-0805, symbol Device:C
- removed C7: NFM21PC105-1uF, Mlab_L:FIR1, symbol SPACEDOS01A_PCB01A-rescue:EMI_Filter_C-device-DATALOGGER01A-rescue-CCP2019V01A-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
- removed D3, D4: LED RED, Mlab_D:LED_1206, symbol Device:LED
- removed R13: 4k7, Mlab_R:SMD-0805, symbol Device:R
- removed R16, R5, R6: 51R, Mlab_R:SMD-0603, symbol Device:R
- removed R7: 22k, Mlab_R:SMD-0805, symbol Device:R
- removed R9: 82R, Mlab_R:SMD-0805, symbol Device:R
- removed U3, U5: SN74LVC1G14-Q1, Package_TO_SOT_SMD:SOT-353_SC-70-5, symbol MLAB_IO:74AHC1G14GV
- removed U8: VCNT2020, Mlab_IO:XDCR_VCNT2020, symbol MLAB_IO:VCNT2020
- added D3: Green 2mA, symbol DATALOGGER01A-rescue:LED-device
- added R5: ?, Mlab_R:SMD-0805, symbol DATALOGGER01A-rescue:R-device
- added U5: VCNT2020, Mlab_IO:XDCR_VCNT2020, symbol MLAB_IO:VCNT2020
- C7: renamed from C8; value 100nF -> 1uF; UST_ID 5c70984712875079b91f8b4c -> (none)
- R10: value 82R -> 4k7; UST_ID 5c70984512875079b91f8976 -> 5c70984612875079b91f8995
- R4: value 470R -> 100R; UST_ID 5c70984512875079b91f8986 -> (none)
- R8: value 22k -> 100R; footprint Mlab_R:SMD-0805 -> Mlab_R:SMD-0603; UST_ID 5c70984712875079b91f8a87 -> (none)
- R9: renamed from R15; value 51R -> 100R; UST_ID 5c70984512875079b91f8953 -> (none)
- renumbered C16 to C10, C12 to C8, C15 to C9, R12 to R11, R11 to R6, R14 to R7, U4 to U3, U6 to U4, U7 to U6
Connections:
- net +3V3: now also R10.1, R11.1, R8.1, R9.1
- net +5V: now also C7.1, U3.1 (VIN), U3.3 (EN); no longer R10.2, R11.1, R8.1
- net COUNT_1: now also R10.2, U4.1 (OSCI), U5.2; no longer R8.2
- net GND: now also D3.2 (A), U5.1, U5.4
- net at U4.2 (OSCO): now also R5.2
- new net: D3.1 (K), R5.1
- new net: R8.2, U5.3
- no-connect marks 2 -> 1
Other:
- moved on the sheet: C10, C6, C9, D2, J1, JP1, R11, R4, R6, R7, R9, U4

Commit message: Edit
Parts:
- C10: UST_ID 5c70984712875079b91f8b4c -> (none)
- C6, C9: UST_ID 5c70984812875079b91f8bbe -> (none)
- C8: UST_ID 5c70984812875079b91f8bc2 -> (none)
- D3: footprint (none) -> LED_SMD:LED_0603_1608Metric
- R10, R11: UST_ID 5c70984612875079b91f8995 -> (none)
- R5: UST_ID 5c70984612875079b91f8990 -> (none)
- R6, R7: UST_ID 5c70984612875079b91f899f -> (none)
Changed lines of the file:
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@@
       (effects (font (size 1.27 1.27)) hide)
     )
-    (property "UST_ID" "5c70984612875079b91f8990" (id 5) (at 114.935 104.775 0)
+    (property "UST_ID" "" (id 5) (at 114.935 104.775 0)
       (effects (font (size 1.27 1.27)) hide)
     )
@@
       (effects (font (size 1.27 1.27)) hide)
     )
-    (property "UST_ID" "5c70984612875079b91f899f" (id 5) (at 155.575 86.995 0)
+    (property "UST_ID" "" (id 5) (at 155.575 86.995 0)
       (effects (font (size 1.27 1.27)) hide)
     )
@@
       (effects (font (size 1.27 1.27)) hide)
     )
-    (property "UST_ID" "5c70984612875079b91f899f" (id 5) (at 161.925 86.995 0)
+    (property "UST_ID" "" (id 5) (at 161.925 86.995 0)
       (effects (font (size 1.27 1.27)) hide)
     )
@@
       (effects (font (size 1.27 1.27)) hide)
     )
-    (property "UST_ID" "5c70984612875079b91f8995" (id 4) (at 266.065 93.98 0)
+    (property "UST_ID" "" (id 4) (at 266.065 93.98 0)
       (effects (font (size 1.27 1.27)) hide)
     )
@@
       (effects (font (size 1.27 1.27)) hide)
     )
-    (property "UST_ID" "5c70984612875079b91f8995" (id 4) (at 266.7 44.45 0)
+    (property "UST_ID" "" (id 4) (at 266.7 44.45 0)
       (effects (font (size 1.27 1.27)) hide)
     )
@@
       (effects (font (size 1.27 1.27)) (justify right))
     )
-    (property "Footprint" "" (id 2) (at 114.935 113.665 0)
+    (property "Footprint" "LED_SMD:LED_0603_1608Metric" (id 2) (at 114.935 113.665 0)
       (effects (font (size 1.27 1.27)) hide)
     )
@@
       (effects (font (size 1.27 1.27)) hide)
     )
-    (property "UST_ID" "5c70984812875079b91f8bbe" (id 4) (at 35.56 177.165 0)
+    (property "UST_ID" "" (id 4) (at 35.56 177.165 0)
       (effects (font (size 1.27 1.27)) hide)
     )
@@
       (effects (font (size 1.27 1.27)) hide)
     )
-    (property "UST_ID" "5c70984812875079b91f8bc2" (id 5) (at 89.535 178.435 0)
+    (property "UST_ID" "" (id 5) (at 89.535 178.435 0)
       (effects (font (size 1.27 1.27)) hide)
     )
@@
       (effects (font (size 1.27 1.27)) hide)
     )
-    (property "UST_ID" "5c70984812875079b91f8bbe" (id 4) (at 109.855 177.165 0)
+    (property "UST_ID" "" (id 4) (at 109.855 177.165 0)
       (effects (font (size 1.27 1.27)) hide)
     )
@@
       (effects (font (size 1.27 1.27)) hide)
     )
-    (property "UST_ID" "5c70984712875079b91f8b4c" (id 4) (at 121.285 177.165 0)
-      (effects (font (size 1.27 1.27)) hide)
-    )
+    (property "UST_ID" "" (id 4) (at 121.285 177.165 0)
+      (effects (font (size 1.27 1.27)) hide)
+    )

Commit message: Edit PCB
Parts:
- removed J2: SM04B-GHS-TB, Connector_JST:JST_GH_SM04B-GHS-TB_1x04-1MP_P1.25mm_Horizontal, symbol MLAB_CONNECTORS_JST:SM04B-GHS-TB
- C10, C7: footprint Mlab_R:SMD-0805 -> Capacitor_SMD:C_0603_1608Metric
- C6, C9: footprint Mlab_R:SMD-0805 -> Capacitor_SMD:C_0805_2012Metric
- C8: footprint Mlab_R:SMD-0603 -> Capacitor_SMD:C_0603_1608Metric
- R10, R11, R4, R5: footprint Mlab_R:SMD-0805 -> Resistor_SMD:R_0603_1608Metric
- R6, R7, R8, R9: footprint Mlab_R:SMD-0603 -> Resistor_SMD:R_0603_1608Metric
Changed lines of the file:
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@@
   (junction (at 161.925 93.345) (diameter 1.016) (color 0 0 0 0))
   (junction (at 169.545 100.965) (diameter 1.016) (color 0 0 0 0))
-  (junction (at 247.015 147.955) (diameter 1.016) (color 0 0 0 0))
   (junction (at 266.065 100.965) (diameter 1.016) (color 0 0 0 0))
   (junction (at 266.7 51.435) (diameter 1.016) (color 0 0 0 0))
@@
     (stroke (width 0) (type solid) (color 0 0 0 0))
   )
-  (wire (pts (xy 243.205 140.335) (xy 248.285 140.335))
-    (stroke (width 0) (type solid) (color 0 0 0 0))
-  )
-  (wire (pts (xy 243.205 142.875) (xy 248.285 142.875))
-    (stroke (width 0) (type solid) (color 0 0 0 0))
-  )
-  (wire (pts (xy 247.015 133.985) (xy 247.015 137.795))
-    (stroke (width 0) (type solid) (color 0 0 0 0))
-  )
-  (wire (pts (xy 247.015 137.795) (xy 248.285 137.795))
-    (stroke (width 0) (type solid) (color 0 0 0 0))
-  )
-  (wire (pts (xy 247.015 145.415) (xy 247.015 147.955))
-    (stroke (width 0) (type solid) (color 0 0 0 0))
-  )
-  (wire (pts (xy 247.015 147.955) (xy 247.015 150.495))
-    (stroke (width 0) (type solid) (color 0 0 0 0))
-  )
-  (wire (pts (xy 248.285 145.415) (xy 247.015 145.415))
-    (stroke (width 0) (type solid) (color 0 0 0 0))
-  )
-  (wire (pts (xy 248.285 147.955) (xy 247.015 147.955))
-    (stroke (width 0) (type solid) (color 0 0 0 0))
-  )
   (wire (pts (xy 258.445 85.725) (xy 260.985 85.725))
     (stroke (width 0) (type solid) (color 0 0 0 0))
@@
   )
   (label "SDA" (at 165.735 95.885 0)
-    (effects (font (size 1.524 1.524)) (justify left bottom))
-  )
-  (label "SCL" (at 243.205 140.335 0)
-    (effects (font (size 1.524 1.524)) (justify left bottom))
-  )
-  (label "SDA" (at 243.205 142.875 0)
     (effects (font (size 1.524 1.524)) (justify left bottom))
   )
@@
     (pin "1")
   )
-  (symbol (lib_id "power:+5V") (at 247.015 133.985 0) (unit 1)
-    (in_bom yes) (on_board yes)
-    (property "Reference" "#PWR035" (id 0) (at 247.015 137.795 0)
-      (effects (font (size 1.27 1.27)) hide)
-    )
-    (property "Value" "+5V" (id 1) (at 247.396 129.5908 0))
-    (property "Footprint" "" (id 2) (at 247.015 133.985 0)
-      (effects (font (size 1.27 1.27)) hide)
-    )
-    (property "Datasheet" "" (id 3) (at 247.015 133.985 0)
-      (effects (font (size 1.27 1.27)) hide)
-    )
-    (pin "1")
-  )
   (symbol (lib_id "power:+3V3") (at 266.065 85.725 0) (unit 1)
     (in_bom yes) (on_board yes)
@@
     (pin "1")
   )
-  (symbol (lib_id "power:GND") (at 247.015 150.495 0) (unit 1)
-    (in_bom yes) (on_board yes)
-    (property "Reference" "#PWR036" (id 0) (at 247.015 156.845 0)
-      (effects (font (size 1.27 1.27)) hide)
-    )
-    (property "Value" "GND" (id 1) (at 247.142 154.8892 0))
-    (property "Footprint" "" (id 2) (at 247.015 150.495 0)
-      (effects (font (size 1.27 1.27)) hide)
-    )
-    (property "Datasheet" "" (id 3) (at 247.015 150.495 0)
-      (effects (font (size 1.27 1.27)) hide)
-    )
-    (pin "1")
-  )
   (symbol (lib_id "power:GND") (at 260.985 86.995 0) (unit 1)
     (in_bom yes) (on_board yes)
@@
     )
     (property "Value" "100R" (id 1) (at 100.965 172.085 90))
-    (property "Footprint" "Mlab_R:SMD-0805" (id 2) (at 100.965 170.307 90)
+    (property "Footprint" "Resistor_SMD:R_0603_1608Metric" (id 2) (at 100.965 170.307 90)
       (effects (font (size 1.27 1.27)) hide)
     )
@@
     (property "Reference" "R5" (id 0) (at 117.475 102.235 90))
     (property "Value" "?" (id 1) (at 114.935 104.775 90))
-    (property "Footprint" "Mlab_R:SMD-0805" (id 2) (at 116.713 104.775 90)
+    (property "Footprint" "Resistor_SMD:R_0603_1608Metric" (id 2) (at 116.713 104.775 90)
       (effects (font (size 1.27 1.27)) hide)
     )
@@
       (effects (font (size 1.27 1.27)) (justify left))
     )
-    (property "Footprint" "Mlab_R:SMD-0603" (id 2) (at 153.797 86.995 90)
+    (property "Footprint" "Resistor_SMD:R_0603_1608Metric" (id 2) (at 153.797 86.995 90)
       (effects (font (size 1.27 1.27)) hide)
     )
@@
       (effects (font (size 1.27 1.27)) (justify left))
     )
-    (property "Footprint" "Mlab_R:SMD-0603" (id 2) (at 160.147 86.995 90)
+    (property "Footprint" "Resistor_SMD:R_0603_1608Metric" (id 2) (at 160.147 86.995 90)
       (effects (font (size 1.27 1.27)) hide)
     )
@@
       (effects (font (size 1.27 1.27)) (justify left))
     )
-    (property "Footprint" "Mlab_R:SMD-0603" (id 2) (at 214.757 80.01 90)
+    (property "Footprint" "Resistor_SMD:R_0603_1608Metric" (id 2) (at 214.757 80.01 90)
       (effects (font (size 1.27 1.27)) hide)
     )
@@
       (effects (font (size 1.27 1.27)) (justify left))
     )
-    (property "Footprint" "Mlab_R:SMD-0603" (id 2) (at 215.392 30.48 90)
+    (property "Footprint" "Resistor_SMD:R_0603_1608Metric" (id 2) (at 215.392 30.48 90)
       (effects (font (size 1.27 1.27)) hide)
     )
@@
       (effects (font (size 1.27 1.27)) (justify left))
     )
-    (property "Footprint" "Mlab_R:SMD-0805" (id 2) (at 264.287 93.98 90)
+    (property "Footprint" "Resistor_SMD:R_0603_1608Metric" (id 2) (at 264.287 93.98 90)
       (effects (font (size 1.27 1.27)) hide)
     )
@@
       (effects (font (size 1.27 1.27)) (justify left))
     )
-    (property "Footprint" "Mlab_R:SMD-0805" (id 2) (at 264.922 44.45 90)
+    (property "Footprint" "Resistor_SMD:R_0603_1608Metric" (id 2) (at 264.922 44.45 90)
       (effects (font (size 1.27 1.27)) hide)
     )
@@
       (effects (font (size 1.27 1.27)) (justify left))
     )
-    (property "Footprint" "Mlab_R:SMD-0805" (id 2) (at 36.5252 180.975 0)
+    (property "Footprint" "Capacitor_SMD:C_0805_2012Metric" (id 2) (at 36.5252 180.975 0)
       (effects (font (size 1.27 1.27)) hide)
     )
@@
       (effects (font (size 1.27 1.27)) (justify left))
     )
-    (property "Footprint" "Mlab_R:SMD-0805" (id 2) (at 48.5902 180.975 0)
+    (property "Footprint" "Capacitor_SMD:C_0603_1608Metric" (id 2) (at 48.5902 180.975 0)
       (effects (font (size 1.27 1.27)) hide)
     )
@@
       (effects (font (size 1.27 1.27)) (justify left))
     )
-    (property "Footprint" "Mlab_R:SMD-0603" (id 2) (at 90.5002 182.245 0)
+    (property "Footprint" "Capacitor_SMD:C_0603_1608Metric" (id 2) (at 90.5002 182.245 0)
       (effects (font (size 1.27 1.27)) hide)
     )
@@
       (effects (font (size 1.27 1.27)) (justify left))
     )
-    (property "Footprint" "Mlab_R:SMD-0805" (id 2) (at 110.8202 180.975 0)
+    (property "Footprint" "Capacitor_SMD:C_0805_2012Metric" (id 2) (at 110.8202 180.975 0)
       (effects (font (size 1.27 1.27)) hide)
     )
@@
       (effects (font (size 1.27 1.27)) (justify left))
     )
-    (property "Footprint" "Mlab_R:SMD-0805" (id 2) (at 122.2502 180.975 0)
+    (property "Footprint" "Capacitor_SMD:C_0603_1608Metric" (id 2) (at 122.2502 180.975 0)
       (effects (font (size 1.27 1.27)) hide)
     )
@@
       (effects (font (size 1.27 1.27)) hide)
     )
-    (pin "1")
-    (pin "2")
-    (pin "3")
-    (pin "4")
-    (pin "MP")
-  )
-  (symbol (lib_id "MLAB_CONNECTORS_JST:SM04B-GHS-TB") (at 253.365 142.875 0) (unit 1)
-    (in_bom yes) (on_board yes)
-    (property "Reference" "J2" (id 0) (at 255.3462 141.3764 0)
-      (effects (font (size 1.524 1.524)) (justify left))
-    )
-    (property "Value" "SM04B-GHS-TB" (id 1) (at 255.3462 144.0942 0)
-      (effects (font (size 1.524 1.524)) (justify left))
-    )
-    (property "Footprint" "Connector_JST:JST_GH_SM04B-GHS-TB_1x04-1MP_P1.25mm_Horizontal" (id 2) (at 253.365 137.795 0)
-      (effects (font (size 1.524 1.524)) hide)
-    )
-    (property "Datasheet" "" (id 3) (at 253.365 137.795 0)
-      (effects (font (size 1.524 1.524)))
-    )
-    (property "UST_id" "" (id 4) (at 253.365 142.875 0)
-      (effects (font (size 1.27 1.27)) hide)
-    )
-    (property "UST_ID" "5c86273d1287500b4e0280be" (id 5) (at 253.365 142.875 0)
-      (effects (font (size 1.27 1.27)) hide)
-    )

Commit message: uprava layoutu, aktualizace elektrod
Parts:
- removed JP1: SolderJumper_3_Bridged12, Jumper:SolderJumper-3_P1.3mm_Bridged12_RoundedPad1.0x1.5mm, symbol Jumper:SolderJumper_3_Bridged12
Connections:
- net GND: now also U4.3 (A0)
Other:
- note added: "Default addr 0x50"
- note removed: "(Edit JP1 for 0x51)"
- note removed: "Default set 0x50"
- note removed: "SET I2C ADRESS"
Changed lines of the file:
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@@
-    (stroke (width 0) (type solid) (color 0 0 0 0))
-  )
-  (wire (pts (xy 89.535 89.535) (xy 89.535 93.345))
     (stroke (width 0) (type solid) (color 0 0 0 0))
   )
@@
     (stroke (width 0) (type solid) (color 0 0 0 0))
   )
-  (wire (pts (xy 92.075 89.535) (xy 89.535 89.535))
-    (stroke (width 0) (type solid) (color 0 0 0 0))
-  )
   (wire (pts (xy 94.615 172.085) (xy 94.615 169.545))
     (stroke (width 0) (type solid) (color 0 0 0 0))
@@
     (stroke (width 0) (type solid) (color 0 0 0 0))
   )
-  (wire (pts (xy 97.155 95.885) (xy 97.155 93.345))
-    (stroke (width 0) (type solid) (color 0 0 0 0))
-  )
-  (wire (pts (xy 97.155 95.885) (xy 120.015 95.885))
-    (stroke (width 0) (type solid) (color 0 0 0 0))
-  )
-  (wire (pts (xy 102.235 84.455) (xy 102.235 89.535))
+  (wire (pts (xy 104.14 95.885) (xy 104.14 96.52))
     (stroke (width 0) (type solid) (color 0 0 0 0))
   )
@@
     (stroke (width 0) (type solid) (color 0 0 0 0))
   )
+  (wire (pts (xy 120.015 95.885) (xy 104.14 95.885))
+    (stroke (width 0) (type solid) (color 0 0 0 0))
+  )
   (wire (pts (xy 121.285 169.545) (xy 121.285 172.085))
     (stroke (width 0) (type solid) (color 0 0 0 0))
@@
     (stroke (width 0) (type solid) (color 0 0 0 0))
   )
-  (text "(Edit JP1 for 0x51)" (at 85.725 79.375 0)
+  (text "Default addr 0x50" (at 86.995 76.835 0)
     (effects (font (size 1.524 1.524)) (justify left bottom))
-  )
-  (text "Default set 0x50" (at 86.995 76.835 0)
-    (effects (font (size 1.524 1.524)) (justify left bottom))
-  )
-  (text "SET I2C ADRESS" (at 106.045 74.295 180)
-    (effects (font (size 1.524 1.524)) (justify right bottom))
   )
   (text "Reflective Optical Sensor" (at 252.095 73.025 180)
@@
     )
     (property "Datasheet" "" (id 3) (at 94.615 169.545 0)
-      (effects (font (size 1.27 1.27)) hide)
-    )
-    (pin "1")
-  )
-  (symbol (lib_id "power:+3V3") (at 102.235 84.455 0) (unit 1)
-    (in_bom yes) (on_board yes)
-    (property "Reference" "#PWR020" (id 0) (at 102.235 88.265 0)
-      (effects (font (size 1.27 1.27)) hide)
-    )
-    (property "Value" "+3V3" (id 1) (at 102.616 80.0608 0))
-    (property "Footprint" "" (id 2) (at 102.235 84.455 0)
-      (effects (font (size 1.27 1.27)) hide)
-    )
-    (property "Datasheet" "" (id 3) (at 102.235 84.455 0)
       (effects (font (size 1.27 1.27)) hide)
     )
@@
     (pin "1")
   )
-  (symbol (lib_id "power:GND") (at 89.535 93.345 0) (unit 1)
-    (in_bom yes) (on_board yes)
-    (property "Reference" "#PWR016" (id 0) (at 89.535 99.695 0)
-      (effects (font (size 1.27 1.27)) hide)
-    )
-    (property "Value" "GND" (id 1) (at 89.662 97.7392 0))
-    (property "Footprint" "" (id 2) (at 89.535 93.345 0)
-      (effects (font (size 1.27 1.27)) hide)
-    )
-    (property "Datasheet" "" (id 3) (at 89.535 93.345 0)
-      (effects (font (size 1.27 1.27)) hide)
-    )
-    (pin "1")
-  )
   (symbol (lib_id "power:GND") (at 89.535 186.055 0) (unit 1)
     (in_bom yes) (on_board yes)
@@
     )
     (property "Datasheet" "" (id 3) (at 89.535 186.055 0)
+      (effects (font (size 1.27 1.27)) hide)
+    )
+    (pin "1")
+  )
+  (symbol (lib_id "power:GND") (at 104.14 96.52 0) (unit 1)
+    (in_bom yes) (on_board yes)
+    (property "Reference" "#PWR016" (id 0) (at 104.14 102.87 0)
+      (effects (font (size 1.27 1.27)) hide)
+    )
+    (property "Value" "GND" (id 1) (at 104.267 100.9142 0))
+    (property "Footprint" "" (id 2) (at 104.14 96.52 0)
+      (effects (font (size 1.27 1.27)) hide)
+    )
+    (property "Datasheet" "" (id 3) (at 104.14 96.52 0)
       (effects (font (size 1.27 1.27)) hide)
     )
@@
     (pin "2")
   )
-  (symbol (lib_id "Jumper:SolderJumper_3_Bridged12") (at 97.155 89.535 0) (unit 1)
-    (in_bom yes) (on_board yes)
-    (property "Reference" "JP1" (id 0) (at 97.155 86.9758 0))
-    (property "Value" "SolderJumper_3_Bridged12" (id 1) (at 97.155 86.735 0)
-      (effects (font (size 1.27 1.27)) hide)
-    )
-    (property "Footprint" "Jumper:SolderJumper-3_P1.3mm_Bridged12_RoundedPad1.0x1.5mm" (id 2) (at 97.155 89.535 0)
-      (effects (font (size 1.27 1.27)) hide)
-    )
-    (property "Datasheet" "~" (id 3) (at 97.155 89.535 0)
-      (effects (font (size 1.27 1.27)) hide)
-    )
-    (pin "1")
-    (pin "2")
-    (pin "3")
-  )
   (symbol (lib_id "MLAB_CONNECTORS_JST:SM04B-GHS-TB") (at 175.895 95.885 0) (unit 1)

Commit message: Uprava PCB
Parts:
- removed D3: Green 2mA, LED_SMD:LED_0603_1608Metric, symbol DATALOGGER01A-rescue:LED-device
- removed R5: ?, Resistor_SMD:R_0603_1608Metric, symbol DATALOGGER01A-rescue:R-device
Connections:
- net COUNT_1_PCFO: now reaches U4.2 (OSCO)
Changed lines of the file:
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@@
-(kicad_sch (version 20210406) (generator eeschema)
+(kicad_sch (version 20210621) (generator eeschema)
   (paper "A4")
   (junction (at 27.94 172.085) (diameter 1.016) (color 0 0 0 0))
@@
     (stroke (width 0) (type solid) (color 0 0 0 0))
   )
-  (wire (pts (xy 114.935 93.345) (xy 114.935 100.965))
-    (stroke (width 0) (type solid) (color 0 0 0 0))
-  )
-  (wire (pts (xy 114.935 109.855) (xy 114.935 108.585))
-    (stroke (width 0) (type solid) (color 0 0 0 0))
-  )
-  (wire (pts (xy 114.935 120.015) (xy 114.935 117.475))
-    (stroke (width 0) (type solid) (color 0 0 0 0))
-  )
   (wire (pts (xy 120.015 93.345) (xy 114.935 93.345))
     (stroke (width 0) (type solid) (color 0 0 0 0))
@@
   )
   (label "COUNT_1" (at 114.935 90.805 180)
+    (effects (font (size 1.27 1.27)) (justify right bottom))
+  )
+  (label "COUNT_1_PCFO" (at 114.935 93.345 180)
     (effects (font (size 1.27 1.27)) (justify right bottom))
   )
@@
     (pin "1")
   )
-  (symbol (lib_id "power:GND") (at 114.935 120.015 0) (unit 1)
-    (in_bom yes) (on_board yes)
-    (property "Reference" "#PWR022" (id 0) (at 114.935 126.365 0)
-      (effects (font (size 1.27 1.27)) hide)
-    )
-    (property "Value" "GND" (id 1) (at 115.062 124.4092 0))
-    (property "Footprint" "" (id 2) (at 114.935 120.015 0)
-      (effects (font (size 1.27 1.27)) hide)
-    )
-    (property "Datasheet" "" (id 3) (at 114.935 120.015 0)
-      (effects (font (size 1.27 1.27)) hide)
-    )
-    (pin "1")
-  )
   (symbol (lib_id "power:GND") (at 121.285 182.245 0) (unit 1)
     (in_bom yes) (on_board yes)
@@
     (pin "2")
   )
-  (symbol (lib_id "DATALOGGER01A-rescue:R-device") (at 114.935 104.775 180) (unit 1)
-    (in_bom yes) (on_board yes)
-    (property "Reference" "R5" (id 0) (at 117.475 102.235 90))
-    (property "Value" "?" (id 1) (at 114.935 104.775 90))
-    (property "Footprint" "Resistor_SMD:R_0603_1608Metric" (id 2) (at 116.713 104.775 90)
-      (effects (font (size 1.27 1.27)) hide)
-    )
-    (property "Datasheet" "" (id 3) (at 114.935 104.775 0)
-      (effects (font (size 1.27 1.27)) hide)
-    )
-    (property "USD_ID" "" (id 4) (at 114.935 104.775 0)
-      (effects (font (size 1.27 1.27)) hide)
-    )
-    (property "UST_ID" "" (id 5) (at 114.935 104.775 0)
-      (effects (font (size 1.27 1.27)) hide)
-    )
-    (pin "1")
-    (pin "2")
-  )
   (symbol (lib_id "Device:R") (at 155.575 86.995 0) (unit 1)
     (in_bom yes) (on_board yes)
@@
       (effects (font (size 1.27 1.27)) hide)
     )
-    (pin "1")
-    (pin "2")
-  )
-  (symbol (lib_id "DATALOGGER01A-rescue:LED-device") (at 114.935 113.665 270) (unit 1)
-    (in_bom yes) (on_board yes)
-    (property "Reference" "D3" (id 0) (at 121.285 112.395 0)
-      (effects (font (size 1.27 1.27)) (justify right))
-    )
-    (property "Value" "Green 2mA" (id 1) (at 118.745 117.475 0)
-      (effects (font (size 1.27 1.27)) (justify right))
-    )
-    (property "Footprint" "LED_SMD:LED_0603_1608Metric" (id 2) (at 114.935 113.665 0)
-      (effects (font (size 1.27 1.27)) hide)
-    )
-    (property "Datasheet" "~" (id 3) (at 114.935 113.665 0)
-      (effects (font (size 1.27 1.27)) hide)
-    )
-    (property "USD_ID" "" (id 4) (at 114.935 113.665 0)
-      (effects (font (size 1.27 1.27)) hide)
-    )
-    (property "UST_ID" "" (id 5) (at 114.935 113.665 0)
-      (effects (font (size 1.27 1.27)) hide)
-    )

Commit message: Edit PCB
Changed lines of the file:
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@@
-(kicad_sch (version 20210621) (generator eeschema)
+(kicad_sch (version 20210406) (generator eeschema)
   (paper "A4")
   (junction (at 27.94 172.085) (diameter 1.016) (color 0 0 0 0))
@@
     (effects (font (size 1.27 1.27)) (justify right bottom))
   )
-  (label "COUNT_1_PCFO" (at 114.935 93.345 180)
-    (effects (font (size 1.27 1.27)) (justify right bottom))
-  )
   (label "SCL" (at 165.735 93.345 0)
     (effects (font (size 1.524 1.524)) (justify left bottom))
@@
     (effects (font (size 1.27 1.27)) (justify left bottom))
   )
-  (label "COUNT_2" (at 269.875 51.435 0)
-    (effects (font (size 1.27 1.27)) (justify left bottom))
+  (global_label "COUNT_1_PCFO" (shape input) (at 114.935 93.345 180) (fields_autoplaced)
+    (effects (font (size 1.27 1.27)) (justify right))
+    (property "Intersheet References" "${INTERSHEET_REFS}" (id 0) (at 98.189 93.2656 0)
+      (effects (font (size 1.27 1.27)) (justify right) hide)
+    )
+  )
+  (global_label "COUNT_2" (shape input) (at 269.875 51.435 0) (fields_autoplaced)
+    (effects (font (size 1.27 1.27)) (justify left))
+    (property "Intersheet References" "${INTERSHEET_REFS}" (id 0) (at 280.6943 51.3556 0)
+      (effects (font (size 1.27 1.27)) (justify left) hide)
+    )
   )
   (symbol (lib_id "power:VCC") (at 89.535 169.545 0) (unit 1)
