File: hw/sch_pcb/USTTHUNDERMILLPCB01A/tachometer.kicad_sch (KiCad schematic)
At the start: 18 parts, among them J1 SM04B-GHS-TB, U3 MIC5504-3.3YM5, U4 PCF8583, U5 VCNT2020, U6 VCNT2020

Commit message: Edit PCB
Parts:
- added C22: 100nF, Capacitor_SMD:C_0603_1608Metric, symbol Device:C
Connections:
- net +3V3: now also C22.1
- net GND: now also C22.2
Changed lines of the file:
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@@
+    (stroke (width 0) (type solid) (color 0 0 0 0))
+  )
+  (wire (pts (xy 82.55 86.36) (xy 82.55 88.9))
+    (stroke (width 0) (type solid) (color 0 0 0 0))
+  )
+  (wire (pts (xy 82.55 96.52) (xy 82.55 97.79))
     (stroke (width 0) (type solid) (color 0 0 0 0))
   )
@@
     (pin "1")
   )
+  (symbol (lib_id "power:+3V3") (at 82.55 86.36 0) (unit 1)
+    (in_bom yes) (on_board yes)
+    (property "Reference" "#PWR0104" (id 0) (at 82.55 90.17 0)
+      (effects (font (size 1.27 1.27)) hide)
+    )
+    (property "Value" "+3V3" (id 1) (at 82.931 81.9658 0))
+    (property "Footprint" "" (id 2) (at 82.55 86.36 0)
+      (effects (font (size 1.27 1.27)) hide)
+    )
+    (property "Datasheet" "" (id 3) (at 82.55 86.36 0)
+      (effects (font (size 1.27 1.27)) hide)
+    )
+    (pin "1")
+  )
   (symbol (lib_id "power:+3V3") (at 94.615 169.545 0) (unit 1)
     (in_bom yes) (on_board yes)
@@
     (pin "1")
   )
+  (symbol (lib_id "power:GND") (at 82.55 97.79 0) (unit 1)
+    (in_bom yes) (on_board yes)
+    (property "Reference" "#PWR0105" (id 0) (at 82.55 104.14 0)
+      (effects (font (size 1.27 1.27)) hide)
+    )
+    (property "Value" "GND" (id 1) (at 82.677 102.1842 0))
+    (property "Footprint" "" (id 2) (at 82.55 97.79 0)
+      (effects (font (size 1.27 1.27)) hide)
+    )
+    (property "Datasheet" "" (id 3) (at 82.55 97.79 0)
+      (effects (font (size 1.27 1.27)) hide)
+    )
+    (pin "1")
+  )
   (symbol (lib_id "power:GND") (at 89.535 186.055 0) (unit 1)
     (in_bom yes) (on_board yes)
@@
       (effects (font (size 1.27 1.27)) hide)
     )
+    (pin "1")
+    (pin "2")
+  )
+  (symbol (lib_id "Device:C") (at 82.55 92.71 0) (unit 1)
+    (in_bom yes) (on_board yes)
+    (property "Reference" "C22" (id 0) (at 85.471 91.5416 0)
+      (effects (font (size 1.27 1.27)) (justify left))
+    )
+    (property "Value" "100nF" (id 1) (at 85.471 93.853 0)
+      (effects (font (size 1.27 1.27)) (justify left))
+    )
+    (property "Footprint" "Capacitor_SMD:C_0603_1608Metric" (id 2) (at 83.5152 96.52 0)
+      (effects (font (size 1.27 1.27)) hide)
+    )
+    (property "Datasheet" "~" (id 3) (at 82.55 92.71 0)
+      (effects (font (size 1.27 1.27)) hide)
+    )
+    (property "UST_ID" "" (id 4) (at 82.55 92.71 0)
+      (effects (font (size 1.27 1.27)) hide)
+    )
