File: hw/sch_pcb/USTTHUNDERMILLPCB01A/tachometer.kicad_sch (KiCad schematic)
At the start: 19 parts, among them J1 SM04B-GHS-TB, U3 MIC5504-3.3YM5, U4 PCF8583, U5 VCNT2020, U6 VCNT2020

Commit message: Edit PCB
Parts:
- C10, C22: UST_ID (none) -> 5c70984812875079b91f8bf2
- C6, C9: UST_ID (none) -> 5c70984812875079b91f8bbe
- C7, C8: UST_ID (none) -> 5c70984812875079b91f8bc2
- R10, R11: UST_ID (none) -> 5c70984512875079b91f8960
- R4, R8, R9: UST_ID (none) -> 5c70984512875079b91f8956
- R6, R7: UST_ID (none) -> 5c70984512875079b91f8962
Changed lines of the file:
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@@
       (effects (font (size 1.27 1.27)) hide)
     )
-    (property "UST_ID" "" (id 4) (at 100.965 172.085 0)
+    (property "UST_ID" "5c70984512875079b91f8956" (id 4) (at 100.965 172.085 0)
       (effects (font (size 1.27 1.27)) hide)
     )
@@
       (effects (font (size 1.27 1.27)) hide)
     )
-    (property "UST_ID" "" (id 5) (at 155.575 86.995 0)
+    (property "UST_ID" "5c70984512875079b91f8962" (id 5) (at 155.575 86.995 0)
       (effects (font (size 1.27 1.27)) hide)
     )
@@
       (effects (font (size 1.27 1.27)) hide)
     )
-    (property "UST_ID" "" (id 5) (at 161.925 86.995 0)
+    (property "UST_ID" "5c70984512875079b91f8962" (id 5) (at 161.925 86.995 0)
       (effects (font (size 1.27 1.27)) hide)
     )
@@
       (effects (font (size 1.27 1.27)) hide)
     )
-    (property "UST_ID" "" (id 4) (at 216.535 80.01 0)
+    (property "UST_ID" "5c70984512875079b91f8956" (id 4) (at 216.535 80.01 0)
       (effects (font (size 1.27 1.27)) hide)
     )
@@
       (effects (font (size 1.27 1.27)) hide)
     )
-    (property "UST_ID" "" (id 4) (at 217.17 30.48 0)
+    (property "UST_ID" "5c70984512875079b91f8956" (id 4) (at 217.17 30.48 0)
       (effects (font (size 1.27 1.27)) hide)
     )
@@
       (effects (font (size 1.27 1.27)) hide)
     )
-    (property "UST_ID" "" (id 4) (at 266.065 93.98 0)
+    (property "UST_ID" "5c70984512875079b91f8960" (id 4) (at 266.065 93.98 0)
       (effects (font (size 1.27 1.27)) hide)
     )
@@
       (effects (font (size 1.27 1.27)) hide)
     )
-    (property "UST_ID" "" (id 4) (at 266.7 44.45 0)
+    (property "UST_ID" "5c70984512875079b91f8960" (id 4) (at 266.7 44.45 0)
       (effects (font (size 1.27 1.27)) hide)
     )
@@
       (effects (font (size 1.27 1.27)) hide)
     )
-    (property "UST_ID" "" (id 4) (at 35.56 177.165 0)
+    (property "UST_ID" "5c70984812875079b91f8bbe" (id 4) (at 35.56 177.165 0)
       (effects (font (size 1.27 1.27)) hide)
     )
@@
       (effects (font (size 1.27 1.27)) hide)
     )
-    (property "UST_ID" "" (id 4) (at 47.625 177.165 0)
+    (property "UST_ID" "5c70984812875079b91f8bc2" (id 4) (at 47.625 177.165 0)
       (effects (font (size 1.27 1.27)) hide)
     )
@@
       (effects (font (size 1.27 1.27)) hide)
     )
-    (property "UST_ID" "" (id 4) (at 82.55 92.71 0)
+    (property "UST_ID" "5c70984812875079b91f8bf2" (id 4) (at 82.55 92.71 0)
       (effects (font (size 1.27 1.27)) hide)
     )
@@
       (effects (font (size 1.27 1.27)) hide)
     )
-    (property "UST_ID" "" (id 5) (at 89.535 178.435 0)
+    (property "UST_ID" "5c70984812875079b91f8bc2" (id 5) (at 89.535 178.435 0)
       (effects (font (size 1.27 1.27)) hide)
     )
@@
       (effects (font (size 1.27 1.27)) hide)
     )
-    (property "UST_ID" "" (id 4) (at 109.855 177.165 0)
+    (property "UST_ID" "5c70984812875079b91f8bbe" (id 4) (at 109.855 177.165 0)
       (effects (font (size 1.27 1.27)) hide)
     )
@@
       (effects (font (size 1.27 1.27)) hide)
     )
-    (property "UST_ID" "" (id 4) (at 121.285 177.165 0)
-      (effects (font (size 1.27 1.27)) hide)
-    )
+    (property "UST_ID" "5c70984812875079b91f8bf2" (id 4) (at 121.285 177.165 0)
+      (effects (font (size 1.27 1.27)) hide)
+    )
